Commit message: In ROS convention x is forward

File: boldbot_description/urdf/boldbot.urdf (robot description, URDF)
Before this commit: robot boldbot, 4 links, 3 joints
Links:
- link torso: geometry visual box size=0.1 0.16 0.101
Joints:
- joint head_tilt_joint: axis 1 0 0 -> 0 1 0

Commit message: Add left arm to URDF model

File: boldbot_description/urdf/boldbot.urdf (robot description, URDF)
Before this commit: robot boldbot, 4 links, 3 joints
Links:
- added link l_lower_arm; visual box size=0.04 0.04 0.06
- added link l_shoulder; visual box size=0.02 0.02 0.02
- added link l_upper_arm; visual box size=0.04 0.04 0.06
Joints:
- added joint l_elbow_joint: type continuous, parent l_upper_arm, child l_lower_arm, origin xyz=0.016 0 -0.06 rpy=0 0 0, axis 0 -1 0
- added joint l_shoulder_pitch_joint: type continuous, parent torso, child l_shoulder, origin xyz=0 0.082 0 rpy=0 0 0, axis 0 1 0
- added joint l_shoulder_roll_joint: type continuous, parent l_shoulder, child l_upper_arm, origin xyz=0 0 -0.016 rpy=0 0 0, axis -1 0 0

Commit message: Add right arm

File: boldbot_description/urdf/boldbot.urdf (robot description, URDF)
Before this commit: robot boldbot, 7 links, 6 joints
Links:
- added link r_lower_arm; visual box size=0.04 0.04 0.06
- added link r_shoulder; visual box size=0.02 0.02 0.02
- added link r_upper_arm; visual box size=0.04 0.04 0.06
- link torso: geometry visual box size=0.1 0.13 0.101
Joints:
- added joint r_elbow_joint: type continuous, parent r_upper_arm, child r_lower_arm, origin xyz=0.016 0 -0.06 rpy=0 0 0, axis 0 -1 0
- added joint r_shoulder_pitch_joint: type continuous, parent torso, child r_shoulder, origin xyz=0 -0.082 0 rpy=0 0 0, axis 0 -1 0
- added joint r_shoulder_roll_joint: type continuous, parent r_shoulder, child r_upper_arm, origin xyz=0 0 -0.016 rpy=0 0 0, axis -1 0 0

Commit message: Add left leg

File: boldbot_description/urdf/boldbot.urdf (robot description, URDF)
Before this commit: robot boldbot, 10 links, 9 joints
Links:
- added link l_ankle; visual box size=0.02 0.02 0.02
- added link l_buttock; visual box size=0.02 0.02 0.02
- added link l_foot; visual box size=0.12 0.05 0.02
- added link l_hip_bracket; visual box size=0.02 0.02 0.02
- added link l_lower_leg; visual box size=0.04 0.04 0.14
- added link l_upper_leg; visual box size=0.04 0.04 0.14
Joints:
- added joint l_ankle_pitch_joint: type continuous, parent l_lower_leg, child l_ankle, origin xyz=0 0 -0.14 rpy=0 0 0, axis 0 1 0
- added joint l_ankle_roll_joint: type continuous, parent l_ankle, child l_foot, origin xyz=0 0 0 rpy=0 0 0, axis 1 0 0
- added joint l_hip_pitch_joint: type continuous, parent l_buttock, child l_upper_leg, origin xyz=0 0 0 rpy=0 0 0, axis 0 -1 0
- added joint l_hip_roll_joint: type continuous, parent l_hip_bracket, child l_buttock, origin xyz=0 0 0 rpy=0 0 0, axis -1 0 0
- added joint l_hip_yaw_joint: type continuous, parent torso, child l_hip_bracket, origin xyz=-0.005 0.037 -0.1222 rpy=0 0 0, axis 0 0 -1
- added joint l_knee_joint: type continuous, parent l_upper_leg, child l_lower_leg, origin xyz=0 0 -0.14 rpy=0 0 0, axis 0 -1 0

Commit message: Add right leg

File: boldbot_description/urdf/boldbot.urdf (robot description, URDF)
Before this commit: robot boldbot, 16 links, 15 joints
Links:
- added link r_ankle; visual box size=0.02 0.02 0.02
- added link r_buttock; visual box size=0.02 0.02 0.02
- added link r_foot; visual box size=0.12 0.05 0.02
- added link r_hip_bracket; visual box size=0.02 0.02 0.02
- added link r_lower_leg; visual box size=0.04 0.04 0.14
- added link r_upper_leg; visual box size=0.04 0.04 0.14
Joints:
- added joint r_ankle_pitch_joint: type continuous, parent r_lower_leg, child r_ankle, origin xyz=0 0 -0.14 rpy=0 0 0, axis 0 -1 0
- added joint r_ankle_roll_joint: type continuous, parent r_ankle, child r_foot, origin xyz=0 0 0 rpy=0 0 0, axis 1 0 0
- added joint r_hip_pitch_joint: type continuous, parent r_buttock, child r_upper_leg, origin xyz=0 0 0 rpy=0 0 0, axis 0 1 0
- added joint r_hip_roll_joint: type continuous, parent r_hip_bracket, child r_buttock, origin xyz=0 0 0 rpy=0 0 0, axis -1 0 0
- added joint r_hip_yaw_joint: type continuous, parent torso, child r_hip_bracket, origin xyz=-0.005 -0.037 -0.1222 rpy=0 0 0, axis 0 0 -1
- added joint r_knee_joint: type continuous, parent r_upper_leg, child r_lower_leg, origin xyz=0 0 -0.14 rpy=0 0 0, axis 0 1 0

Commit message: Better size torso

File: boldbot_description/urdf/boldbot.urdf (robot description, URDF)
Before this commit: robot boldbot, 22 links, 21 joints
Links:
- link torso: geometry visual box size=0.1 0.13 0.17

Commit message: using boldhumanoid json names

File: boldbot_description/urdf/boldbot.urdf (robot description, URDF)
Before this commit: robot boldbot, 22 links, 21 joints
Links:
- removed link l_ankle
- removed link l_buttock
- removed link l_foot
- removed link l_hip_bracket
- removed link l_lower_arm
- removed link l_lower_leg
- removed link l_shoulder
- removed link l_upper_arm
- removed link l_upper_leg
- removed link r_ankle
- removed link r_buttock
- removed link r_foot
- removed link r_hip_bracket
- removed link r_lower_arm
- removed link r_lower_leg
- removed link r_shoulder
- removed link r_upper_arm
- removed link r_upper_leg
- added link ankle-l; visual box size=0.02 0.02 0.02
- added link ankle-r; visual box size=0.02 0.02 0.02
- added link buttock-l; visual box size=0.02 0.02 0.02
- added link buttock-r; visual box size=0.02 0.02 0.02
- added link foot-l; visual box size=0.12 0.05 0.02
- added link foot-r; visual box size=0.12 0.05 0.02
- added link hip-bracket-l; visual box size=0.02 0.02 0.02
- added link hip-bracket-r; visual box size=0.02 0.02 0.02
- added link lower-arm-l; visual box size=0.04 0.04 0.06
- added link lower-arm-r; visual box size=0.04 0.04 0.06
- added link lower-leg-l; visual box size=0.04 0.04 0.14
- added link lower-leg-r; visual box size=0.04 0.04 0.14
- added link shoulder-l; visual box size=0.02 0.02 0.02
- added link shoulder-r; visual box size=0.02 0.02 0.02
- added link upper-arm-l; visual box size=0.04 0.04 0.06
- added link upper-arm-r; visual box size=0.04 0.04 0.06
- added link upper-leg-l; visual box size=0.04 0.04 0.14
- added link upper-leg-r; visual box size=0.04 0.04 0.14
Joints:
- removed joint head_pan_joint
- removed joint head_tilt_joint
- removed joint l_ankle_pitch_joint
- removed joint l_ankle_roll_joint
- removed joint l_elbow_joint
- removed joint l_hip_pitch_joint
- removed joint l_hip_roll_joint
- removed joint l_hip_yaw_joint
- removed joint l_knee_joint
- removed joint l_shoulder_pitch_joint
- removed joint l_shoulder_roll_joint
- removed joint r_ankle_pitch_joint
- removed joint r_ankle_roll_joint
- removed joint r_elbow_joint
- removed joint r_hip_pitch_joint
- removed joint r_hip_roll_joint
- removed joint r_hip_yaw_joint
- removed joint r_knee_joint
- removed joint r_shoulder_pitch_joint
- removed joint r_shoulder_roll_joint
- added joint ankle-pitch-l: type continuous, parent lower-leg-l, child ankle-l, origin xyz=0 0 -0.14 rpy=0 0 0, axis 0 1 0
- added joint ankle-pitch-r: type continuous, parent lower-leg-r, child ankle-r, origin xyz=0 0 -0.14 rpy=0 0 0, axis 0 -1 0
- added joint ankle-roll-l: type continuous, parent ankle-l, child foot-l, origin xyz=0 0 0 rpy=0 0 0, axis 1 0 0
- added joint ankle-roll-r: type continuous, parent ankle-r, child foot-r, origin xyz=0 0 0 rpy=0 0 0, axis 1 0 0
- added joint elbow-l: type continuous, parent upper-arm-l, child lower-arm-l, origin xyz=0.016 0 -0.06 rpy=0 0 0, axis 0 -1 0
- added joint elbow-r: type continuous, parent upper-arm-r, child lower-arm-r, origin xyz=0.016 0 -0.06 rpy=0 0 0, axis 0 -1 0
- added joint head-pan: type continuous, parent torso, child neck, origin xyz=0 0 0.0505 rpy=0 0 0, axis 0 0 1
- added joint head-tilt: type continuous, parent neck, child head, origin xyz=0 0 0 rpy=0 0 0, axis 0 1 0
- added joint hip-pitch-l: type continuous, parent buttock-l, child upper-leg-l, origin xyz=0 0 0 rpy=0 0 0, axis 0 -1 0
- added joint hip-pitch-r: type continuous, parent buttock-r, child upper-leg-r, origin xyz=0 0 0 rpy=0 0 0, axis 0 1 0
- added joint hip-roll-l: type continuous, parent hip-bracket-l, child buttock-l, origin xyz=0 0 0 rpy=0 0 0, axis -1 0 0
- added joint hip-roll-r: type continuous, parent hip-bracket-r, child buttock-r, origin xyz=0 0 0 rpy=0 0 0, axis -1 0 0
- added joint hip-yaw-l: type continuous, parent torso, child hip-bracket-l, origin xyz=-0.005 0.037 -0.1222 rpy=0 0 0, axis 0 0 -1
- added joint hip-yaw-r: type continuous, parent torso, child hip-bracket-r, origin xyz=-0.005 -0.037 -0.1222 rpy=0 0 0, axis 0 0 -1
- added joint knee-l: type continuous, parent upper-leg-l, child lower-leg-l, origin xyz=0 0 -0.14 rpy=0 0 0, axis 0 -1 0
- added joint knee-r: type continuous, parent upper-leg-r, child lower-leg-r, origin xyz=0 0 -0.14 rpy=0 0 0, axis 0 1 0
- added joint shoulder-pitch-l: type continuous, parent torso, child shoulder-l, origin xyz=0 0.082 0 rpy=0 0 0, axis 0 1 0
- added joint shoulder-pitch-r: type continuous, parent torso, child shoulder-r, origin xyz=0 -0.082 0 rpy=0 0 0, axis 0 -1 0
- added joint shoulder-roll-l: type continuous, parent shoulder-l, child upper-arm-l, origin xyz=0 0 -0.016 rpy=0 0 0, axis -1 0 0
- added joint shoulder-roll-r: type continuous, parent shoulder-r, child upper-arm-r, origin xyz=0 0 -0.016 rpy=0 0 0, axis -1 0 0

Commit message: Fix some joint orientations

File: boldbot_description/urdf/boldbot.urdf (robot description, URDF)
Before this commit: robot boldbot, 22 links, 21 joints
Joints:
- joint elbow-l: axis 0 -1 0 -> 0 1 0; origin xyz=0.016 0 -0.06 rpy=0 0 0 -> xyz=0.016 0 -0.06 rpy=0 -1.570796327 0
- joint elbow-r: origin xyz=0.016 0 -0.06 rpy=0 0 0 -> xyz=0.016 0 -0.06 rpy=0 -1.570796327 0
- joint head-tilt: axis 0 1 0 -> 0 -1 0; origin xyz=0 0 0 rpy=0 0 0 -> xyz=0 0 0 rpy=0 0.785398163 0
- joint shoulder-roll-l: origin xyz=0 0 -0.016 rpy=0 0 0 -> xyz=0 0 -0.016 rpy=0.785398163 0 0
- joint shoulder-roll-r: origin xyz=0 0 -0.016 rpy=0 0 0 -> xyz=0 0 -0.016 rpy=-0.785398163 0 0

Commit message: Add inertia to all links, so they show up in Gazebo

File: boldbot_description/urdf/boldbot.urdf (robot description, URDF)
Before this commit: robot boldbot, 22 links, 21 joints
Links:
- link ankle-l: mass None -> 0.1
- link ankle-r: mass None -> 0.1
- link buttock-l: mass None -> 0.1
- link buttock-r: mass None -> 0.1
- link foot-l: mass None -> 0.1
- link foot-r: mass None -> 0.1
- link head: mass None -> .2; geometry collision box size=0.03 0.03 0.06; visual box size=0.03 0.03 0.06
- link hip-bracket-l: mass None -> .1
- link hip-bracket-r: mass None -> 0.1
- link lower-arm-l: mass None -> 0.1
- link lower-arm-r: mass None -> 0.1
- link lower-leg-l: mass None -> 0.1
- link lower-leg-r: mass None -> 0.1
- link neck: mass None -> 0.1
- link shoulder-l: mass None -> 0.1
- link shoulder-r: mass None -> 0.1
- link torso: mass None -> 1; geometry collision box size=0.1 0.13 0.17; visual box size=0.1 0.13 0.17
- link upper-arm-l: mass None -> 0.1
- link upper-arm-r: mass None -> .1
- link upper-leg-l: mass None -> 0.1
- link upper-leg-r: mass None -> 0.1

Commit message: Add collision tags

File: boldbot_description/urdf/boldbot.urdf (robot description, URDF)
Before this commit: robot boldbot, 22 links, 21 joints
Links:
- link foot-l: geometry collision box size=0.12 0.05 0.02; visual box size=0.12 0.05 0.02
- link foot-r: geometry collision box size=0.12 0.05 0.02; visual box size=0.12 0.05 0.02
- link lower-arm-l: geometry collision box size=0.04 0.04 0.06; visual box size=0.04 0.04 0.06
- link lower-arm-r: geometry collision box size=0.04 0.04 0.06; visual box size=0.04 0.04 0.06
- link lower-leg-l: geometry collision box size=0.04 0.04 0.14; visual box size=0.04 0.04 0.14
- link lower-leg-r: geometry collision box size=0.04 0.04 0.14; visual box size=0.04 0.04 0.14
- link upper-arm-l: geometry collision box size=0.04 0.04 0.06; visual box size=0.04 0.04 0.06
- link upper-arm-r: geometry collision box size=0.04 0.04 0.06; visual box size=0.04 0.04 0.06
- link upper-leg-l: geometry collision box size=0.04 0.04 0.14; visual box size=0.04 0.04 0.14
- link upper-leg-r: geometry collision box size=0.04 0.04 0.14; visual box size=0.04 0.04 0.14
