Commit message: Start of adding MX28s through xacro

File: boldbot_description/urdf/boldbot.urdf.xacro (robot description, xacro)
@@ -1,4 +1,23 @@
 <?xml version="1.0" ?>
-<robot name="boldbot">
+<robot name="boldbot" xmlns:xacro="http://www.ros.org/wiki/xacro">
+  <xacro:macro name="mx28" params="name">
+    <link name="${name}">
+      <visual>
+        <geometry>
+          <mesh filename="/home/sander/src/boldbot/boldbot_description/meshes/mx28.stl" scale="0.001 0.001 0.001" />
+        </geometry>
+      </visual>
+      <collision>
+        <geometry>
+          <mesh filename="/home/sander/src/boldbot/boldbot_description/meshes/mx28.stl" scale="0.001 0.001 0.001" />
+        </geometry>
+      </collision>
+      <inertial>
+        <origin xyz="0 0 0" />
+        <mass value="0.072"/>
+        <inertia ixx="0.02292366"  ixy="0.0"  ixz="0.0" iyy="0.01516566" iyz="0.0" izz="0.02296632" />
+      </inertial>
+    </link>
+  </xacro:macro>
   <!-- dummy first link, directly connects with torso -->
   <link name="base_link" />
@@ -10,26 +29,33 @@
   <link name="torso">
     <visual>
-      <origin rpy="0 0 0" xyz="0 0 -0.035" />
-      <geometry>
-        <box size="0.1 0.13 0.17"/>
-      </geometry>
-    </visual>
-    <collision>
-      <origin rpy="0 0 0" xyz="0 0 -0.035" />
-      <geometry>
-        <box size="0.1 0.13 0.17"/>
-      </geometry>
-    </collision>
-    <inertial>
-      <origin xyz="0 0 0" />
-      <mass value="1"/>
-      <inertia ixx="1e-3"  ixy="0.0"  ixz="0.0" iyy="1e-3" iyz="0.0" izz="1e-3" />
-    </inertial>
-  </link>
-  <joint name="head-pan" type="continuous">
+      <origin rpy="0 0 0" xyz="0 0 0" />
+      <geometry>
+        <box size="0.109 0.1 0.045"/>
+      </geometry>
+    </visual>
+    <collision>
+      <origin rpy="0 0 0" xyz="0 0 0" />
+      <geometry>
+        <box size="0.109 0.1 0.045"/>
+      </geometry>
+    </collision>
+    <inertial>
+      <origin xyz="0 0 0" />
+      <mass value="0.1"/>
+      <inertia ixx="1e-3"  ixy="0.0"  ixz="0.0" iyy="1e-3" iyz="0.0" izz="1e-3" />
+    </inertial>
+  </link>
+  <joint name="torso-mx28-neck" type="fixed">
     <parent link="torso" />
+    <child link="mx28-neck" />
+    <origin rpy="0 0 3.141592654" xyz="0.02 0 0.045" />
+  </joint>
+  <xacro:mx28 name="mx28-neck"/>
+  <joint name="head-pan" type="revolute">
+    <parent link="mx28-neck" />
     <child link="neck" />
     <origin rpy="0 0 0" xyz="0 0 0.0505" />
     <axis xyz="0 0 1" />
+    <limit effort="2.8" velocity="5.6548668" lower="-2.6179939" upper="2.6179939" />
   </joint>
   <link name="neck">
@@ -51,4 +77,5 @@
     <origin rpy="0 0.785398163 0" xyz="0 0 0" />
     <axis xyz="0 -1 0" />
+    <limit effort="2.8" velocity="5.6548668" lower="-2.6179939" upper="2.6179939" />
   </joint>
   <link name="head">
@@ -77,4 +104,5 @@
     <origin rpy="0 0 0" xyz="0 0.082 0" />
     <axis xyz="0 1 0" />
+    <limit effort="2.8" velocity="5.6548668" lower="-2.6179939" upper="2.6179939" />
   </joint>
   <link name="shoulder-l">
@@ -96,4 +124,5 @@
     <origin rpy="0.785398163 0 0" xyz="0 0 -0.016" />
     <axis xyz="-1 0 0" />
+    <limit effort="2.8" velocity="5.6548668" lower="-2.6179939" upper="2.6179939" />
   </joint>
   <link name="upper-arm-l">
@@ -121,4 +150,5 @@
     <origin rpy="0 -1.570796327 0" xyz="0.016 0 -0.06" />
     <axis xyz="0 1 0" />
+    <limit effort="2.8" velocity="5.6548668" lower="-2.6179939" upper="2.6179939" />
   </joint>
   <link name="lower-arm-l">
@@ -147,4 +177,5 @@
     <origin rpy="0 0 0" xyz="0 -0.082 0" />
     <axis xyz="0 -1 0" />
+    <limit effort="2.8" velocity="5.6548668" lower="-2.6179939" upper="2.6179939" />
   </joint>
   <link name="shoulder-r">
@@ -166,4 +197,5 @@
     <origin rpy="-0.785398163 0 0" xyz="0 0 -0.016" />
     <axis xyz="-1 0 0" />
+    <limit effort="2.8" velocity="5.6548668" lower="-2.6179939" upper="2.6179939" />
   </joint>
   <link name="upper-arm-r">
@@ -191,4 +223,5 @@
     <origin rpy="0 -1.570796327 0" xyz="0.016 0 -0.06" />
     <axis xyz="0 -1 0" />
+    <limit effort="2.8" velocity="5.6548668" lower="-2.6179939" upper="2.6179939" />
   </joint>
   <link name="lower-arm-r">
@@ -217,4 +250,5 @@
     <origin rpy="0 0 0" xyz="-0.005 0.037 -0.1222" />
     <axis xyz="0 0 -1" />
+    <limit effort="2.8" velocity="5.6548668" lower="-2.6179939" upper="2.6179939" />
   </joint>
   <link name="hip-bracket-l">
@@ -236,4 +270,5 @@
     <origin rpy="0 0 0" xyz="0 0 0" />
     <axis xyz="-1 0 0" />
+    <limit effort="2.8" velocity="5.6548668" lower="-2.6179939" upper="2.6179939" />
   </joint>
   <link name="buttock-l">
@@ -255,4 +290,5 @@
     <origin rpy="0 0 0" xyz="0 0 0" />
     <axis xyz="0 -1 0" />
+    <limit effort="2.8" velocity="5.6548668" lower="-2.6179939" upper="2.6179939" />
   </joint>
   <link name="upper-leg-l">
@@ -280,4 +316,5 @@
     <origin rpy="0 0 0" xyz="0 0 -0.14" />
     <axis xyz="0 -1 0" />
+    <limit effort="2.8" velocity="5.6548668" lower="-2.6179939" upper="2.6179939" />
   </joint>
   <link name="lower-leg-l">
@@ -305,4 +342,5 @@
     <origin rpy="0 0 0" xyz="0 0 -0.14" />
     <axis xyz="0 1 0" />
+    <limit effort="2.8" velocity="5.6548668" lower="-2.6179939" upper="2.6179939" />
   </joint>
   <link name="ankle-l">
@@ -324,4 +362,5 @@
     <origin rpy="0 0 0" xyz="0 0 0" />
     <axis xyz="1 0 0" />
+    <limit effort="2.8" velocity="5.6548668" lower="-2.6179939" upper="2.6179939" />
   </joint>
   <link name="foot-l">
@@ -350,4 +389,5 @@
     <origin rpy="0 0 0" xyz="-0.005 -0.037 -0.1222" />
     <axis xyz="0 0 -1" />
+    <limit effort="2.8" velocity="5.6548668" lower="-2.6179939" upper="2.6179939" />
   </joint>
   <link name="hip-bracket-r">
@@ -369,4 +409,5 @@
     <origin rpy="0 0 0" xyz="0 0 0" />
     <axis xyz="-1 0 0" />
+    <limit effort="2.8" velocity="5.6548668" lower="-2.6179939" upper="2.6179939" />
   </joint>
   <link name="buttock-r">
@@ -388,4 +429,5 @@
     <origin rpy="0 0 0" xyz="0 0 0" />
     <axis xyz="0 1 0" />
+    <limit effort="2.8" velocity="5.6548668" lower="-2.6179939" upper="2.6179939" />
   </joint>
   <link name="upper-leg-r">
@@ -413,4 +455,5 @@
     <origin rpy="0 0 0" xyz="0 0 -0.14" />
     <axis xyz="0 1 0" />
+    <limit effort="2.8" velocity="5.6548668" lower="-2.6179939" upper="2.6179939" />
   </joint>
   <link name="lower-leg-r">
@@ -438,4 +481,5 @@
     <origin rpy="0 0 0" xyz="0 0 -0.14" />
     <axis xyz="0 -1 0" />
+    <limit effort="2.8" velocity="5.6548668" lower="-2.6179939" upper="2.6179939" />
   </joint>
   <link name="ankle-r">
@@ -457,4 +501,5 @@
     <origin rpy="0 0 0" xyz="0 0 0" />
     <axis xyz="1 0 0" />
+    <limit effort="2.8" velocity="5.6548668" lower="-2.6179939" upper="2.6179939" />
   </joint>
   <link name="foot-r">

Commit message: Head and left arm

File: boldbot_description/urdf/boldbot.urdf.xacro (robot description, xacro)
@@ -1,12 +1,17 @@
 <?xml version="1.0" ?>
 <robot name="boldbot" xmlns:xacro="http://www.ros.org/wiki/xacro">
-  <xacro:macro name="mx28" params="name">
+  <xacro:macro name="mx28" params="name xyz rpy">
     <link name="${name}">
       <visual>
+        <origin xyz="${xyz}" rpy="${rpy}" />
         <geometry>
           <mesh filename="/home/sander/src/boldbot/boldbot_description/meshes/mx28.stl" scale="0.001 0.001 0.001" />
         </geometry>
+        <material name="DarkGrey">
+          <color rgba="0.20 0.20 0.20 1.0"/>
+        </material>
       </visual>
       <collision>
+        <origin xyz="${xyz}" rpy="${rpy}" />
         <geometry>
           <mesh filename="/home/sander/src/boldbot/boldbot_description/meshes/mx28.stl" scale="0.001 0.001 0.001" />
@@ -14,9 +19,12 @@
       </collision>
       <inertial>
-        <origin xyz="0 0 0" />
+        <origin xyz="${xyz}" rpy="${rpy}" />
         <mass value="0.072"/>
-        <inertia ixx="0.02292366"  ixy="0.0"  ixz="0.0" iyy="0.01516566" iyz="0.0" izz="0.02296632" />
+        <inertia ixx="0.00002292366"  ixy="0.0"  ixz="0.0" iyy="0.00001516566" iyz="0.0" izz="0.00002296632" />
       </inertial>
     </link>
+    <gazebo reference="${name}">
+      <material>Gazebo/Grey</material>
+    </gazebo>
   </xacro:macro>
   <!-- dummy first link, directly connects with torso -->
@@ -31,29 +39,29 @@
       <origin rpy="0 0 0" xyz="0 0 0" />
       <geometry>
-        <box size="0.109 0.1 0.045"/>
-      </geometry>
-    </visual>
-    <collision>
-      <origin rpy="0 0 0" xyz="0 0 0" />
-      <geometry>
-        <box size="0.109 0.1 0.045"/>
-      </geometry>
-    </collision>
-    <inertial>
-      <origin xyz="0 0 0" />
-      <mass value="0.1"/>
-      <inertia ixx="1e-3"  ixy="0.0"  ixz="0.0" iyy="1e-3" iyz="0.0" izz="1e-3" />
-    </inertial>
-  </link>
-  <joint name="torso-mx28-neck" type="fixed">
+        <box size="0.1 0.109 0.045"/>
+      </geometry>
+    </visual>
+    <collision>
+      <origin rpy="0 0 0" xyz="0 0 0" />
+      <geometry>
+        <box size="0.1 0.109 0.045"/>
+      </geometry>
+    </collision>
+    <inertial>
+      <origin xyz="0 0 0" />
+      <mass value="0.1"/>
+      <inertia ixx="1e-3"  ixy="0.0"  ixz="0.0" iyy="1e-3" iyz="0.0" izz="1e-3" />
+    </inertial>
+  </link>
+  <joint name="torso-mx28-head-pan" type="fixed">
     <parent link="torso" />
-    <child link="mx28-neck" />
-    <origin rpy="0 0 3.141592654" xyz="0.02 0 0.045" />
-  </joint>
-  <xacro:mx28 name="mx28-neck"/>
+    <child link="mx28-head-pan" />
+    <origin rpy="0 0 0" xyz="0.02 0 0.045" />
+  </joint>
+  <xacro:mx28 name="mx28-head-pan" xyz="0 0 0" rpy="0 0 3.141592654"/>
   <joint name="head-pan" type="revolute">
-    <parent link="mx28-neck" />
+    <parent link="mx28-head-pan" />
     <child link="neck" />
-    <origin rpy="0 0 0" xyz="0 0 0.0505" />
+    <origin rpy="0 0 0" xyz="0 0 0" />
     <axis xyz="0 0 1" />
     <limit effort="2.8" velocity="5.6548668" lower="-2.6179939" upper="2.6179939" />
@@ -61,33 +69,39 @@
   <link name="neck">
     <visual>
-      <origin rpy="0 0 0" xyz="0 0 0" />
-      <geometry>
-        <box size="0.02 0.02 0.02"/>
-      </geometry>
-    </visual>
-    <inertial>
-      <origin xyz="0 0 0" />
-      <mass value="0.1"/>
-      <inertia ixx="1e-4"  ixy="0.0"  ixz="0.0" iyy="1e-4" iyz="0.0" izz="1e-4" />
-    </inertial>
-  </link>
-  <joint name="head-tilt" type="continuous">
+      <origin rpy="0 0 0" xyz="0 0 0.03" />
+      <geometry>
+        <box size="0.01 0.01 0.01"/>
+      </geometry>
+    </visual>
+    <inertial>
+      <origin xyz="0 0 0" />
+      <mass value="1e-3"/>
+      <inertia ixx="1e-4"  ixy="0.0"  ixz="0.0" iyy="1e-4" iyz="0.0" izz="1e-4" />
+    </inertial>
+  </link>
+  <joint name="head-tilt" type="revolute">
     <parent link="neck" />
+    <child link="mx28-head-tilt" />
+    <origin xyz="0 0 0.05" />
+    <axis xyz="0 1 0" />
+    <limit effort="2.8" velocity="5.6548668" lower="-2.6179939" upper="2.6179939" />
+  </joint>
+  <xacro:mx28 name="mx28-head-tilt" xyz="0 0 0" rpy="0 -1.570796327 -1.570796327"/>
+  <joint name="head-tilt-head" type="fixed">
+    <parent link="mx28-head-tilt" />
     <child link="head" />
-    <origin rpy="0 0.785398163 0" xyz="0 0 0" />
-    <axis xyz="0 -1 0" />
-    <limit effort="2.8" velocity="5.6548668" lower="-2.6179939" upper="2.6179939" />
+    <origin rpy="0 0 0" xyz="0 0 0.065" />
   </joint>
   <link name="head">
     <visual>
-      <origin rpy="0 0 0" xyz="0 0 0.03"/>
-      <geometry>
-        <box size="0.03 0.03 0.06" />
-      </geometry>
-    </visual>
-    <collision>
-      <origin rpy="0 0 0" xyz="0 0 0.03"/>
-      <geometry>
-        <box size="0.03 0.03 0.06" />
+      <origin rpy="0 0 0" xyz="0 0 0"/>
+      <geometry>
+        <box size="0.05 0.1 0.04" />
+      </geometry>
+    </visual>
+    <collision>
+      <origin rpy="0 0 0" xyz="0 0 0"/>
+      <geometry>
+        <box size="0.05 0.1 0.04" />
       </geometry>
     </collision>
@@ -99,8 +113,14 @@
   </link>
   <!-- Left Arm -->
-  <joint name="shoulder-pitch-l" type="continuous">
+  <joint name="torso-mx28-shoulder-pitch-l" type="fixed">
     <parent link="torso" />
+    <child link="mx28-shoulder-pitch-l" />
+    <origin xyz="0.02 0.04 0.045" />
+  </joint>
+  <xacro:mx28 name="mx28-shoulder-pitch-l" xyz="0 0 0" rpy="1.570796327 0 3.141592654"/>
+  <joint name="shoulder-pitch-l" type="revolute">
+    <parent link="mx28-shoulder-pitch-l" />
     <child link="shoulder-l" />
-    <origin rpy="0 0 0" xyz="0 0.082 0" />
+    <origin rpy="0 0 0" xyz="0 0 0" />
     <axis xyz="0 1 0" />
     <limit effort="2.8" velocity="5.6548668" lower="-2.6179939" upper="2.6179939" />
@@ -108,45 +128,33 @@
   <link name="shoulder-l">
     <visual>
-      <origin rpy="0 0 0" xyz="0 0 0" />
-      <geometry>
-        <box size="0.02 0.02 0.02"/>
-      </geometry>
-    </visual>
-    <inertial>
-      <origin xyz="0 0 0" />
-      <mass value="0.1"/>
-      <inertia ixx="1e-4"  ixy="0.0"  ixz="0.0" iyy="1e-4" iyz="0.0" izz="1e-4" />
-    </inertial>
-  </link>
-  <joint name="shoulder-roll-l" type="continuous">
+      <origin rpy="0 0 0" xyz="0 0.021 -0.008" />
+      <geometry>
+        <box size="0.01 0.01 0.01"/>
+      </geometry>
+    </visual>
+    <inertial>
+      <origin xyz="0 0 0" />
+      <mass value="0.1"/>
+      <inertia ixx="1e-4"  ixy="0.0"  ixz="0.0" iyy="1e-4" iyz="0.0" izz="1e-4" />
+    </inertial>
+  </link>
+  <joint name="shoulder-roll-l" type="revolute">
     <parent link="shoulder-l" />
-    <child link="upper-arm-l" />
-    <origin rpy="0.785398163 0 0" xyz="0 0 -0.016" />
+    <child link="mx28-shoulder-roll-l" />
+    <origin rpy="0.785398163 0 0" xyz="0 0.042 -0.016" />
     <axis xyz="-1 0 0" />
     <limit effort="2.8" velocity="5.6548668" lower="-2.6179939" upper="2.6179939" />
   </joint>
-  <link name="upper-arm-l">
-    <visual>
-      <origin rpy="0 0 0" xyz="0 0 -0.03" />
-      <geometry>
-        <box size="0.04 0.04 0.06"/>
-      </geometry>
-    </visual>
-    <collision>
-      <origin rpy="0 0 0" xyz="0 0 -0.03" />
-      <geometry>
-        <box size="0.04 0.04 0.06"/>
-      </geometry>
-    </collision>
-    <inertial>
-      <origin xyz="0 0 0" />
-      <mass value="0.1"/>
-      <inertia ixx="1e-3"  ixy="0.0"  ixz="0.0" iyy="1e-3" iyz="0.0" izz="1e-3" />
-    </inertial>
-  </link>
-  <joint name="elbow-l" type="continuous">
-    <parent link="upper-arm-l" />
+  <xacro:mx28 name="mx28-shoulder-roll-l" xyz="0 0 0" rpy="0 1.570796327 0"/>
+  <joint name="mx28-shoulder-roll-l-mx28-elbow-l" type="fixed">
+    <parent link="mx28-shoulder-roll-l" />
+    <child link="mx28-elbow-l" />
+    <origin xyz="0.016 0 -0.06" />
+  </joint>
+  <xacro:mx28 name="mx28-elbow-l" xyz="0 0 0" rpy="1.570796327 0 3.141592654"/>
+  <joint name="elbow-l" type="revolute">
+    <parent link="mx28-elbow-l" />
     <child link="lower-arm-l" />
-    <origin rpy="0 -1.570796327 0" xyz="0.016 0 -0.06" />
+    <origin xyz="0 0 0" rpy="0 0 0"/>
     <axis xyz="0 1 0" />
     <limit effort="2.8" velocity="5.6548668" lower="-2.6179939" upper="2.6179939" />
@@ -154,13 +162,13 @@
   <link name="lower-arm-l">
     <visual>
-      <origin rpy="0 0 0" xyz="-0.016 0 -0.03" />
-      <geometry>
-        <box size="0.04 0.04 0.06"/>
-      </geometry>
-    </visual>
-    <collision>
-      <origin rpy="0 0 0" xyz="-0.016 0 -0.03" />
-      <geometry>
-        <box size="0.04 0.04 0.06"/>
+      <origin rpy="1.570796327 0 0" xyz="0.055 0.02 -0.02" />
+      <geometry>
+        <mesh filename="/home/sander/src/boldbot/boldbot_description/meshes/armcover.stl" scale="0.001 0.001 0.001"/>
+      </geometry>
+    </visual>
+    <collision>
+      <origin rpy="1.570796327 0 0" xyz="0.055 0.02 -0.02" />
+      <geometry>
+        <mesh filename="/home/sander/src/boldbot/boldbot_description/meshes/armcover.stl" scale="0.001 0.001 0.001"/>
       </geometry>
     </collision>
@@ -172,4 +180,10 @@
   </link>
   <!-- Right Arm -->
+  <joint name="torso-mx28-shoulder-pitch-r" type="fixed">
+    <parent link="torso" />
+    <child link="mx28-shoulder-pitch-r" />
+    <origin xyz="0.02 -0.04 0.045" />
+  </joint>
+  <xacro:mx28 name="mx28-shoulder-pitch-r" xyz="0 0 0" rpy="-1.570796327 0 3.141592654"/>
   <joint name="shoulder-pitch-r" type="continuous">
     <parent link="torso" />
