Commit message: Right arm through using xacro

File: boldbot_description/urdf/boldbot.urdf.xacro (robot description, xacro)
@@ -112,150 +112,76 @@
     </inertial>
   </link>
-  <!-- Left Arm -->
-  <joint name="torso-mx28-shoulder-pitch-l" type="fixed">
-    <parent link="torso" />
-    <child link="mx28-shoulder-pitch-l" />
-    <origin xyz="0.02 0.04 0.045" />
-  </joint>
-  <xacro:mx28 name="mx28-shoulder-pitch-l" xyz="0 0 0" rpy="1.570796327 0 3.141592654"/>
-  <joint name="shoulder-pitch-l" type="revolute">
-    <parent link="mx28-shoulder-pitch-l" />
-    <child link="shoulder-l" />
-    <origin rpy="0 0 0" xyz="0 0 0" />
-    <axis xyz="0 1 0" />
-    <limit effort="2.8" velocity="5.6548668" lower="-2.6179939" upper="2.6179939" />
-  </joint>
-  <link name="shoulder-l">
-    <visual>
-      <origin rpy="0 0 0" xyz="0 0.021 -0.008" />
-      <geometry>
-        <box size="0.01 0.01 0.01"/>
-      </geometry>
-    </visual>
-    <inertial>
-      <origin xyz="0 0 0" />
-      <mass value="0.1"/>
-      <inertia ixx="1e-4"  ixy="0.0"  ixz="0.0" iyy="1e-4" iyz="0.0" izz="1e-4" />
-    </inertial>
-  </link>
-  <joint name="shoulder-roll-l" type="revolute">
-    <parent link="shoulder-l" />
-    <child link="mx28-shoulder-roll-l" />
-    <origin rpy="0.785398163 0 0" xyz="0 0.042 -0.016" />
-    <axis xyz="-1 0 0" />
-    <limit effort="2.8" velocity="5.6548668" lower="-2.6179939" upper="2.6179939" />
-  </joint>
-  <xacro:mx28 name="mx28-shoulder-roll-l" xyz="0 0 0" rpy="0 1.570796327 0"/>
-  <joint name="mx28-shoulder-roll-l-mx28-elbow-l" type="fixed">
-    <parent link="mx28-shoulder-roll-l" />
-    <child link="mx28-elbow-l" />
-    <origin xyz="0.016 0 -0.06" />
-  </joint>
-  <xacro:mx28 name="mx28-elbow-l" xyz="0 0 0" rpy="1.570796327 0 3.141592654"/>
-  <joint name="elbow-l" type="revolute">
-    <parent link="mx28-elbow-l" />
-    <child link="lower-arm-l" />
-    <origin xyz="0 0 0" rpy="0 0 0"/>
-    <axis xyz="0 1 0" />
-    <limit effort="2.8" velocity="5.6548668" lower="-2.6179939" upper="2.6179939" />
-  </joint>
-  <link name="lower-arm-l">
-    <visual>
-      <origin rpy="1.570796327 0 0" xyz="0.055 0.02 -0.02" />
-      <geometry>
-        <mesh filename="/home/sander/src/boldbot/boldbot_description/meshes/armcover.stl" scale="0.001 0.001 0.001"/>
-      </geometry>
-    </visual>
-    <collision>
-      <origin rpy="1.570796327 0 0" xyz="0.055 0.02 -0.02" />
-      <geometry>
-        <mesh filename="/home/sander/src/boldbot/boldbot_description/meshes/armcover.stl" scale="0.001 0.001 0.001"/>
-      </geometry>
-    </collision>
-    <inertial>
-      <origin xyz="0 0 0" />
-      <mass value="0.1"/>
-      <inertia ixx="1e-3"  ixy="0.0"  ixz="0.0" iyy="1e-3" iyz="0.0" izz="1e-3" />
-    </inertial>
-  </link>
-  <!-- Right Arm -->
-  <joint name="torso-mx28-shoulder-pitch-r" type="fixed">
-    <parent link="torso" />
-    <child link="mx28-shoulder-pitch-r" />
-    <origin xyz="0.02 -0.04 0.045" />
-  </joint>
-  <xacro:mx28 name="mx28-shoulder-pitch-r" xyz="0 0 0" rpy="-1.570796327 0 3.141592654"/>
-  <joint name="shoulder-pitch-r" type="continuous">
-    <parent link="torso" />
-    <child link="shoulder-r" />
-    <origin rpy="0 0 0" xyz="0 -0.082 0" />
-    <axis xyz="0 -1 0" />
-    <limit effort="2.8" velocity="5.6548668" lower="-2.6179939" upper="2.6179939" />
-  </joint>
-  <link name="shoulder-r">
-    <visual>
-      <origin rpy="0 0 0" xyz="0 0 0" />
-      <geometry>
-        <box size="0.02 0.02 0.02"/>
-      </geometry>
-    </visual>
-    <inertial>
-      <origin xyz="0 0 0" />
-      <mass value="0.1"/>
-      <inertia ixx="1e-4"  ixy="0.0"  ixz="0.0" iyy="1e-4" iyz="0.0" izz="1e-4" />
-    </inertial>
-  </link>
-  <joint name="shoulder-roll-r" type="continuous">
-    <parent link="shoulder-r" />
-    <child link="upper-arm-r" />
-    <origin rpy="-0.785398163 0 0" xyz="0 0 -0.016" />
-    <axis xyz="-1 0 0" />
-    <limit effort="2.8" velocity="5.6548668" lower="-2.6179939" upper="2.6179939" />
-  </joint>
-  <link name="upper-arm-r">
-    <visual>
-      <origin rpy="0 0 0" xyz="0 0 -0.03" />
-      <geometry>
-        <box size="0.04 0.04 0.06"/>
-      </geometry>
-    </visual>
-    <collision>
-      <origin rpy="0 0 0" xyz="0 0 -0.03" />
-      <geometry>
-        <box size="0.04 0.04 0.06"/>
-      </geometry>
-    </collision>
-    <inertial>
-      <origin xyz="0 0 0" />
-      <mass value=".1"/>
-      <inertia ixx="1e-3"  ixy="0.0"  ixz="0.0" iyy="1e-3" iyz="0.0" izz="1e-3" />
-    </inertial>
-  </link>
-  <joint name="elbow-r" type="continuous">
-    <parent link="upper-arm-r" />
-    <child link="lower-arm-r" />
-    <origin rpy="0 -1.570796327 0" xyz="0.016 0 -0.06" />
-    <axis xyz="0 -1 0" />
-    <limit effort="2.8" velocity="5.6548668" lower="-2.6179939" upper="2.6179939" />
-  </joint>
-  <link name="lower-arm-r">
-    <visual>
-      <origin rpy="0 0 0" xyz="-0.016 0 -0.03" />
-      <geometry>
-        <box size="0.04 0.04 0.06"/>
-      </geometry>
-    </visual>
-    <collision>
-      <origin rpy="0 0 0" xyz="-0.016 0 -0.03" />
-      <geometry>
-        <box size="0.04 0.04 0.06"/>
-      </geometry>
-    </collision>
-    <inertial>
-      <origin xyz="0 0 0" />
-      <mass value="0.1"/>
-      <inertia ixx="1e-3"  ixy="0.0"  ixz="0.0" iyy="1e-3" iyz="0.0" izz="1e-3" />
-    </inertial>
-  </link>
+  <!-- Arms -->
+  <xacro:macro name="arm" params="side">
+    <xacro:property name="lr" value="${1 if side == 'l' else -1}" />
+    <joint name="torso-mx28-shoulder-pitch-${side}" type="fixed">
+      <parent link="torso" />
+      <child link="mx28-shoulder-pitch-${side}" />
+      <origin xyz="0.02 ${lr * 0.04} 0.045" />
+    </joint>
+    <xacro:mx28 name="mx28-shoulder-pitch-${side}" xyz="0 0 0" rpy="${lr * 1.570796327} 0 3.141592654"/>
+    <joint name="shoulder-pitch-${side}" type="revolute">
+      <parent link="mx28-shoulder-pitch-${side}" />
+      <child link="shoulder-${side}" />
+      <origin rpy="0 0 0" xyz="0 0 0" />
+      <axis xyz="0 ${lr} 0" />
+      <limit effort="2.8" velocity="5.6548668" lower="-2.6179939" upper="2.6179939" />
+    </joint>
+    <link name="shoulder-${side}">
+      <visual>
+        <origin rpy="0 0 0" xyz="0 ${lr * 0.021} -0.008" />
+        <geometry>
+          <box size="0.01 0.01 0.01"/>
+        </geometry>
+      </visual>
+      <inertial>
+        <origin xyz="0 0 0" />
+        <mass value="0.1"/>
+        <inertia ixx="1e-4"  ixy="0.0"  ixz="0.0" iyy="1e-4" iyz="0.0" izz="1e-4" />
+      </inertial>
+    </link>
+    <joint name="shoulder-roll-${side}" type="revolute">
+      <parent link="shoulder-${side}" />
+      <child link="mx28-shoulder-roll-${side}" />
+      <origin xyz="0 ${lr * 0.042} -0.016" rpy="${lr * 0.785398163} 0 0" />
+      <axis xyz="1 0 0" />
+      <limit effort="2.8" velocity="5.6548668" lower="-2.6179939" upper="2.6179939" />
+    </joint>
+    <xacro:mx28 name="mx28-shoulder-roll-${side}" xyz="0 0 0" rpy="0 1.570796327 0"/>
+    <joint name="mx28-shoulder-roll-${side}-mx28-elbow-${side}" type="fixed">
+      <parent link="mx28-shoulder-roll-${side}" />
+      <child link="mx28-elbow-${side}" />
+      <origin xyz="0.016 0 -0.06" />
+    </joint>
+    <xacro:mx28 name="mx28-elbow-${side}" xyz="0 0 0" rpy="${lr * 1.570796327} 0 3.141592654"/>
+    <joint name="elbow-${side}" type="revolute">
+      <parent link="mx28-elbow-${side}" />
+      <child link="lower-arm-${side}" />
+      <origin xyz="0 0 0" rpy="0 0 0"/>
+      <axis xyz="0 ${lr} 0" />
+      <limit effort="2.8" velocity="5.6548668" lower="-2.6179939" upper="2.6179939" />
+    </joint>
+    <link name="lower-arm-${side}">
+      <visual>
+        <origin xyz="0.055 ${lr * 0.02} -0.02" rpy="${lr * 1.570796327} 0 0" />
+        <geometry>
+          <mesh filename="/home/sander/src/boldbot/boldbot_description/meshes/armcover.stl" scale="0.001 0.001 0.001"/>
+        </geometry>
+      </visual>
+      <collision>
+        <origin rpy="1.570796327 0 0" xyz="0.055 0.02 -0.02" />
+        <geometry>
+          <mesh filename="/home/sander/src/boldbot/boldbot_description/meshes/armcover.stl" scale="0.001 0.001 0.001"/>
+        </geometry>
+      </collision>
+      <inertial>
+        <origin xyz="0 0 0" />
+        <mass value="0.1"/>
+        <inertia ixx="1e-3"  ixy="0.0"  ixz="0.0" iyy="1e-3" iyz="0.0" izz="1e-3" />
+      </inertial>
+    </link>
+  </xacro:macro>
+  <xacro:arm side="l"/>
+  <xacro:arm side="r"/>
   <!-- Left Leg -->
   <joint name="hip-yaw-l" type="continuous">

Commit message: Add legs macros and selfCollide

File: boldbot_description/urdf/boldbot.urdf.xacro (robot description, xacro)
@@ -25,5 +25,6 @@
     </link>
     <gazebo reference="${name}">
-      <material>Gazebo/Grey</material>
+      <material>Gazebo/DarkGrey</material>
+      <selfCollide>true</selfCollide>
     </gazebo>
   </xacro:macro>
@@ -54,4 +55,8 @@
     </inertial>
   </link>
+  <gazebo reference="torso">
+    <material>Gazebo/Grey</material>
+    <selfCollide>true</selfCollide>
+  </gazebo>
   <joint name="torso-mx28-head-pan" type="fixed">
     <parent link="torso" />
@@ -112,4 +117,8 @@
     </inertial>
   </link>
+  <gazebo reference="head">
+    <material>Gazebo/Grey</material>
+    <selfCollide>true</selfCollide>
+  </gazebo>
   <!-- Arms -->
   <xacro:macro name="arm" params="side">
@@ -170,5 +179,5 @@
       </visual>
       <collision>
-        <origin rpy="1.570796327 0 0" xyz="0.055 0.02 -0.02" />
+        <origin xyz="0.055 ${lr * 0.02} -0.02" rpy="${lr * 1.570796327} 0 0" />
         <geometry>
           <mesh filename="/home/sander/src/boldbot/boldbot_description/meshes/armcover.stl" scale="0.001 0.001 0.001"/>
@@ -181,284 +190,160 @@
       </inertial>
     </link>
+    <gazebo reference="lower-arm-${side}">
+      <material>Gazebo/Grey</material>
+      <selfCollide>true</selfCollide>
+    </gazebo>
   </xacro:macro>
   <xacro:arm side="l"/>
   <xacro:arm side="r"/>
   <!-- Left Leg -->
-  <joint name="hip-yaw-l" type="continuous">
-    <parent link="torso" />
-    <child link="hip-bracket-l" />
-    <origin rpy="0 0 0" xyz="-0.005 0.037 -0.1222" />
-    <axis xyz="0 0 -1" />
-    <limit effort="2.8" velocity="5.6548668" lower="-2.6179939" upper="2.6179939" />
-  </joint>
-  <link name="hip-bracket-l">
-    <visual>
+  <xacro:macro name="leg" params="side">
+    <xacro:property name="lr" value="${1 if side == 'l' else -1}"/>
+    <joint name="torso-mx28-hip-yaw-${side}" type="fixed">
+      <parent link="torso" />
+      <child link="mx28-hip-yaw-${side}" />
+      <origin xyz="0.018 ${lr * 0.037} -0.04" />
+    </joint>
+    <xacro:mx28 name="mx28-hip-yaw-${side}" xyz="0 0 0" rpy="${lr * 3.141592654} 0 3.141592654"/>
+    <joint name="hip-yaw-${side}" type="continuous">
+      <parent link="mx28-hip-yaw-${side}" />
+      <child link="hip-bracket-${side}" />
       <origin rpy="0 0 0" xyz="0 0 0" />
-      <geometry>
-        <box size="0.02 0.02 0.02"/>
-      </geometry>
-    </visual>
-    <inertial>
-      <origin xyz="0 0 0" />
-      <mass value=".1"/>
-      <inertia ixx="1e-4"  ixy="0.0"  ixz="0.0" iyy="1e-4" iyz="0.0" izz="1e-4" />
-    </inertial>
-  </link>
-  <joint name="hip-roll-l" type="continuous">
-    <parent link="hip-bracket-l" />
-    <child link="buttock-l" />
-    <origin rpy="0 0 0" xyz="0 0 0" />
-    <axis xyz="-1 0 0" />
-    <limit effort="2.8" velocity="5.6548668" lower="-2.6179939" upper="2.6179939" />
-  </joint>
-  <link name="buttock-l">
-    <visual>
-      <origin rpy="0 0 0" xyz="0 0 0" />
-      <geometry>
-        <box size="0.02 0.02 0.02"/>
-      </geometry>
-    </visual>
-    <inertial>
-      <origin xyz="0 0 0" />
-      <mass value="0.1"/>
-      <inertia ixx="1e-4"  ixy="0.0"  ixz="0.0" iyy="1e-4" iyz="0.0" izz="1e-4" />
-    </inertial>
-  </link>
-  <joint name="hip-pitch-l" type="continuous">
-    <parent link="buttock-l" />
-    <child link="upper-leg-l" />
-    <origin rpy="0 0 0" xyz="0 0 0" />
-    <axis xyz="0 -1 0" />
-    <limit effort="2.8" velocity="5.6548668" lower="-2.6179939" upper="2.6179939" />
-  </joint>
-  <link name="upper-leg-l">
-    <visual>
-      <origin rpy="0 0 0" xyz="0 0 -0.07" />
-      <geometry>
-        <box size="0.04 0.04 0.14"/>
-      </geometry>
-    </visual>
-    <collision>
-      <origin rpy="0 0 0" xyz="0 0 -0.07" />
-      <geometry>
-        <box size="0.04 0.04 0.14"/>
-      </geometry>
-    </collision>
-    <inertial>
-      <origin xyz="0 0 0" />
-      <mass value="0.1"/>
-      <inertia ixx="1e-3"  ixy="0.0"  ixz="0.0" iyy="1e-3" iyz="0.0" izz="1e-3" />
-    </inertial>
-  </link>
-  <joint name="knee-l" type="continuous">
-    <parent link="upper-leg-l" />
-    <child link="lower-leg-l" />
-    <origin rpy="0 0 0" xyz="0 0 -0.14" />
-    <axis xyz="0 -1 0" />
-    <limit effort="2.8" velocity="5.6548668" lower="-2.6179939" upper="2.6179939" />
-  </joint>
-  <link name="lower-leg-l">
-    <visual>
-      <origin rpy="0 0 0" xyz="0 0 -0.07" />
-      <geometry>
-        <box size="0.04 0.04 0.14"/>
-      </geometry>
-    </visual>
-    <collision>
-      <origin rpy="0 0 0" xyz="0 0 -0.07" />
-      <geometry>
-        <box size="0.04 0.04 0.14"/>
-      </geometry>
-    </collision>
-    <inertial>
-      <origin xyz="0 0 0" />
-      <mass value="0.1"/>
-      <inertia ixx="1e-3"  ixy="0.0"  ixz="0.0" iyy="1e-3" iyz="0.0" izz="1e-3" />
-    </inertial>
-  </link>
-  <joint name="ankle-pitch-l" type="continuous">
-    <parent link="lower-leg-l" />
-    <child link="ankle-l" />
-    <origin rpy="0 0 0" xyz="0 0 -0.14" />
-    <axis xyz="0 1 0" />
-    <limit effort="2.8" velocity="5.6548668" lower="-2.6179939" upper="2.6179939" />
-  </joint>
-  <link name="ankle-l">
-    <visual>
-      <origin rpy="0 0 0" xyz="0 0 0" />
-      <geometry>
-        <box size="0.02 0.02 0.02"/>
-      </geometry>
-    </visual>
-    <inertial>
-      <origin xyz="0 0 0" />
-      <mass value="0.1"/>
-      <inertia ixx="1e-4"  ixy="0.0"  ixz="0.0" iyy="1e-4" iyz="0.0" izz="1e-4" />
-    </inertial>
-  </link>
-  <joint name="ankle-roll-l" type="continuous">
-    <parent link="ankle-l" />
-    <child link="foot-l" />
-    <origin rpy="0 0 0" xyz="0 0 0" />
-    <axis xyz="1 0 0" />
-    <limit effort="2.8" velocity="5.6548668" lower="-2.6179939" upper="2.6179939" />
-  </joint>
-  <link name="foot-l">
-    <visual>
-      <origin rpy="0 0 0" xyz="0 0 -0.0335" />
-      <geometry>
-        <box size="0.12 0.05 0.02"/>
-      </geometry>
-    </visual>
-    <collision>
-      <origin rpy="0 0 0" xyz="0 0 -0.0335" />
-      <geometry>
-        <box size="0.12 0.05 0.02"/>
-      </geometry>
-    </collision>
-    <inertial>
-      <origin xyz="0 0 0" />
-      <mass value="0.1"/>
-      <inertia ixx="1e-3"  ixy="0.0"  ixz="0.0" iyy="1e-3" iyz="0.0" izz="1e-3" />
-    </inertial>
-  </link>
-  <!-- Right Leg -->
-  <joint name="hip-yaw-r" type="continuous">
-    <parent link="torso" />
-    <child link="hip-bracket-r" />
-    <origin rpy="0 0 0" xyz="-0.005 -0.037 -0.1222" />
-    <axis xyz="0 0 -1" />
-    <limit effort="2.8" velocity="5.6548668" lower="-2.6179939" upper="2.6179939" />
-  </joint>
-  <link name="hip-bracket-r">
-    <visual>
-      <origin rpy="0 0 0" xyz="0 0 0" />
-      <geometry>
-        <box size="0.02 0.02 0.02"/>
-      </geometry>
-    </visual>
-    <inertial>
-      <origin xyz="0 0 0" />
-      <mass value="0.1"/>
-      <inertia ixx="1e-4"  ixy="0.0"  ixz="0.0" iyy="1e-4" iyz="0.0" izz="1e-4" />
-    </inertial>
-  </link>
-  <joint name="hip-roll-r" type="continuous">
-    <parent link="hip-bracket-r" />
-    <child link="buttock-r" />
-    <origin rpy="0 0 0" xyz="0 0 0" />
-    <axis xyz="-1 0 0" />
-    <limit effort="2.8" velocity="5.6548668" lower="-2.6179939" upper="2.6179939" />
-  </joint>
-  <link name="buttock-r">
-    <visual>
-      <origin rpy="0 0 0" xyz="0 0 0" />
-      <geometry>
-        <box size="0.02 0.02 0.02"/>
-      </geometry>
-    </visual>
-    <inertial>
-      <origin xyz="0 0 0" />
-      <mass value="0.1"/>
-      <inertia ixx="1e-4"  ixy="0.0"  ixz="0.0" iyy="1e-4" iyz="0.0" izz="1e-4" />
-    </inertial>
-  </link>
-  <joint name="hip-pitch-r" type="continuous">
-    <parent link="buttock-r" />
-    <child link="upper-leg-r" />
-    <origin rpy="0 0 0" xyz="0 0 0" />
-    <axis xyz="0 1 0" />
-    <limit effort="2.8" velocity="5.6548668" lower="-2.6179939" upper="2.6179939" />
-  </joint>
-  <link name="upper-leg-r">
-    <visual>
-      <origin rpy="0 0 0" xyz="0 0 -0.07" />
-      <geometry>
-        <box size="0.04 0.04 0.14"/>
-      </geometry>
-    </visual>
-    <collision>
-      <origin rpy="0 0 0" xyz="0 0 -0.07" />
-      <geometry>
-        <box size="0.04 0.04 0.14"/>
-      </geometry>
-    </collision>
-    <inertial>
-      <origin xyz="0 0 0" />
-      <mass value="0.1"/>
-      <inertia ixx="1e-3"  ixy="0.0"  ixz="0.0" iyy="1e-3" iyz="0.0" izz="1e-3" />
-    </inertial>
-  </link>
-  <joint name="knee-r" type="continuous">
-    <parent link="upper-leg-r" />
-    <child link="lower-leg-r" />
-    <origin rpy="0 0 0" xyz="0 0 -0.14" />
-    <axis xyz="0 1 0" />
-    <limit effort="2.8" velocity="5.6548668" lower="-2.6179939" upper="2.6179939" />
-  </joint>
-  <link name="lower-leg-r">
-    <visual>
-      <origin rpy="0 0 0" xyz="0 0 -0.07" />
-      <geometry>
-        <box size="0.04 0.04 0.14"/>
-      </geometry>
-    </visual>
-    <collision>
-      <origin rpy="0 0 0" xyz="0 0 -0.07" />
-      <geometry>
-        <box size="0.04 0.04 0.14"/>
-      </geometry>
-    </collision>
-    <inertial>
-      <origin xyz="0 0 0" />
-      <mass value="0.1"/>
-      <inertia ixx="1e-3"  ixy="0.0"  ixz="0.0" iyy="1e-3" iyz="0.0" izz="1e-3" />
-    </inertial>
-  </link>
-  <joint name="ankle-pitch-r" type="continuous">
-    <parent link="lower-leg-r" />
-    <child link="ankle-r" />
-    <origin rpy="0 0 0" xyz="0 0 -0.14" />
-    <axis xyz="0 -1 0" />
-    <limit effort="2.8" velocity="5.6548668" lower="-2.6179939" upper="2.6179939" />
-  </joint>
-  <link name="ankle-r">
-    <visual>
-      <origin rpy="0 0 0" xyz="0 0 0" />
-      <geometry>
-        <box size="0.02 0.02 0.02"/>
-      </geometry>
-    </visual>
-    <inertial>
-      <origin xyz="0 0 0" />
-      <mass value="0.1"/>
-      <inertia ixx="1e-4"  ixy="0.0"  ixz="0.0" iyy="1e-4" iyz="0.0" izz="1e-4" />
-    </inertial>
-  </link>
-  <joint name="ankle-roll-r" type="continuous">
-    <parent link="ankle-r" />
-    <child link="foot-r" />
-    <origin rpy="0 0 0" xyz="0 0 0" />
-    <axis xyz="1 0 0" />
-    <limit effort="2.8" velocity="5.6548668" lower="-2.6179939" upper="2.6179939" />
-  </joint>
-  <link name="foot-r">
-    <visual>
-      <origin rpy="0 0 0" xyz="0 0 -0.0335" />
-      <geometry>
-        <box size="0.12 0.05 0.02"/>
-      </geometry>
-    </visual>
-    <collision>
-      <origin rpy="0 0 0" xyz="0 0 -0.0335" />
-      <geometry>
-        <box size="0.12 0.05 0.02"/>
-      </geometry>
-    </collision>
-    <inertial>
-      <origin xyz="0 0 0" />
-      <mass value="0.1"/>
-      <inertia ixx="1e-4"  ixy="0.0"  ixz="0.0" iyy="1e-4" iyz="0.0" izz="1e-4" />
-    </inertial>
-  </link>
+      <axis xyz="0 0 -1" />
+      <limit effort="2.8" velocity="5.6548668" lower="-2.6179939" upper="2.6179939" />
+    </joint>
+    <link name="hip-bracket-${side}">
+      <inertial>
+        <origin xyz="0 0 0" />
+        <mass value=".1"/>
+        <inertia ixx="1e-4"  ixy="0.0"  ixz="0.0" iyy="1e-4" iyz="0.0" izz="1e-4" />
+      </inertial>
+    </link>
+    <joint name="hip-roll-${side}" type="continuous">
+      <parent link="hip-bracket-${side}" />
+      <child link="mx28-hip-roll-${side}" />
+      <origin rpy="0 0 0" xyz="-0.05 0 -0.04" /> <!-- TODO: guessed -->
+      <axis xyz="-1 0 0" />
+      <limit effort="2.8" velocity="5.6548668" lower="-2.6179939" upper="2.6179939" />
+    </joint>
+    <xacro:mx28 name="mx28-hip-roll-${side}" xyz="0 0 0" rpy="0 1.570796327 0"/>
+    <joint name="mx28-hip-roll-mx28-hip-pitch-${side}" type="fixed">
+      <parent link="mx28-hip-roll-${side}" />
+      <child link="mx28-hip-pitch-${side}" />
+      <origin xyz="0.05 0 0" rpy="0 0 0" />
+    </joint>
+    <xacro:mx28 name="mx28-hip-pitch-${side}" xyz="0 0 0" rpy="1.570796327 1.570796327 0"/>
+    <joint name="mx28-hip-pitch-upper-leg-${side}" type="continuous">
+      <parent link="mx28-hip-pitch-${side}" />
+      <child link="upper-leg-${side}" />
+      <origin xyz="0 0 0" rpy="0 0 0" />
+      <axis xyz="0 -1 0" />
+      <limit effort="2.8" velocity="5.6548668" lower="-2.6179939" upper="2.6179939" />
+    </joint>
+    <link name="upper-leg-${side}">
+      <visual>
+        <origin xyz="0 0 0" rpy="0 1.570796327 0" />
+        <geometry>
+          <mesh filename="/home/sander/src/boldbot/boldbot_description/meshes/thigh.stl" scale="0.001 0.001 0.001"/>
+        </geometry>
+      </visual>
+      <collision>
+        <origin xyz="0 0 0" rpy="0 1.570796327 0" />
+        <geometry>
+          <mesh filename="/home/sander/src/boldbot/boldbot_description/meshes/thigh.stl" scale="0.001 0.001 0.001"/>
+        </geometry>
+      </collision>
+      <inertial>
+        <origin xyz="0 0 0" />
+        <mass value="0.1"/>
+        <inertia ixx="1e-3"  ixy="0.0"  ixz="0.0" iyy="1e-3" iyz="0.0" izz="1e-3" />
+      </inertial>
+    </link>
+    <gazebo reference="upper-leg-${side}">
+      <material>Gazebo/Grey</material>
+      <selfCollide>true</selfCollide>
+    </gazebo>
+    <joint name="upper-leg-mx28-knee-${side}" type="fixed">
+      <parent link="upper-leg-${side}" />
+      <child link="mx28-knee-${side}" />
+      <origin xyz="0 0 -0.143" rpy="0 0 0" />
+    </joint>
+    <xacro:mx28 name="mx28-knee-${side}" xyz="0 0 0" rpy="1.570796327 -1.570796327 0"/>
+    <joint name="mx28-knee-lower-leg-${side}" type="continuous">
+      <parent link="mx28-knee-${side}" />
+      <child link="lower-leg-${side}" />
+      <origin xyz="0 0 0" rpy="0 0 0" />
+      <axis xyz="0 -1 0" />
+      <limit effort="2.8" velocity="5.6548668" lower="-2.6179939" upper="2.6179939" />
+    </joint>
+    <link name="lower-leg-${side}">
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