Commit message: Use find to locat meshes rather than hardcoded path

File: boldbot_description/urdf/boldbot.urdf.xacro (robot description, xacro)
@@ -6,5 +6,5 @@
         <origin xyz="${xyz}" rpy="${rpy}" />
         <geometry>
-          <mesh filename="/home/sander/src/boldbot/boldbot_description/meshes/mx28.stl" scale="0.001 0.001 0.001" />
+          <mesh filename="$(find boldbot_description)/meshes/mx28.stl" scale="0.001 0.001 0.001" />
         </geometry>
         <material name="DarkGrey">
@@ -15,5 +15,5 @@
         <origin xyz="${xyz}" rpy="${rpy}" />
         <geometry>
-          <mesh filename="/home/sander/src/boldbot/boldbot_description/meshes/mx28.stl" scale="0.001 0.001 0.001" />
+          <mesh filename="$(find boldbot_description)/meshes/mx28.stl" scale="0.001 0.001 0.001" />
         </geometry>
       </collision>
@@ -175,5 +175,5 @@
         <origin xyz="0.055 ${lr * 0.02} -0.02" rpy="${lr * 1.570796327} 0 0" />
         <geometry>
-          <mesh filename="/home/sander/src/boldbot/boldbot_description/meshes/armcover.stl" scale="0.001 0.001 0.001"/>
+          <mesh filename="$(find boldbot_description)/meshes/armcover.stl" scale="0.001 0.001 0.001"/>
         </geometry>
       </visual>
@@ -181,5 +181,5 @@
         <origin xyz="0.055 ${lr * 0.02} -0.02" rpy="${lr * 1.570796327} 0 0" />
         <geometry>
-          <mesh filename="/home/sander/src/boldbot/boldbot_description/meshes/armcover.stl" scale="0.001 0.001 0.001"/>
+          <mesh filename="$(find boldbot_description)/meshes/armcover.stl" scale="0.001 0.001 0.001"/>
         </geometry>
       </collision>
@@ -245,5 +245,5 @@
         <origin xyz="0 0 0" rpy="0 1.570796327 0" />
         <geometry>
-          <mesh filename="/home/sander/src/boldbot/boldbot_description/meshes/thigh.stl" scale="0.001 0.001 0.001"/>
+          <mesh filename="$(find boldbot_description)/meshes/thigh.stl" scale="0.001 0.001 0.001"/>
         </geometry>
       </visual>
@@ -251,5 +251,5 @@
         <origin xyz="0 0 0" rpy="0 1.570796327 0" />
         <geometry>
-          <mesh filename="/home/sander/src/boldbot/boldbot_description/meshes/thigh.stl" scale="0.001 0.001 0.001"/>
+          <mesh filename="$(find boldbot_description)/meshes/thigh.stl" scale="0.001 0.001 0.001"/>
         </geometry>
       </collision>
@@ -281,5 +281,5 @@
         <origin xyz="0.0175 0 -0.019" rpy="3.141592654 1.570796327 0" />
         <geometry>
-          <mesh filename="/home/sander/src/boldbot/boldbot_description/meshes/shin.stl" scale="0.001 0.001 0.001"/>
+          <mesh filename="$(find boldbot_description)/meshes/shin.stl" scale="0.001 0.001 0.001"/>
         </geometry>
       </visual>
@@ -287,5 +287,5 @@
         <origin xyz="0.0175 0 -0.019" rpy="3.141592654 1.570796327 0" />
         <geometry>
-          <mesh filename="/home/sander/src/boldbot/boldbot_description/meshes/shin.stl" scale="0.001 0.001 0.001"/>
+          <mesh filename="$(find boldbot_description)/meshes/shin.stl" scale="0.001 0.001 0.001"/>
         </geometry>
       </collision>
@@ -325,5 +325,5 @@
         <origin xyz="0.05 ${lr * 0.01} -0.02" rpy="0 0 -1.570796327" /> <!-- TODO: guessed y offset -->
         <geometry>
-          <mesh filename="/home/sander/src/boldbot/boldbot_description/meshes/nicefoot${side}.stl" scale="0.001 0.001 0.001"/>
+          <mesh filename="$(find boldbot_description)/meshes/nicefoot${side}.stl" scale="0.001 0.001 0.001"/>
         </geometry>
       </visual>
@@ -331,5 +331,5 @@
         <origin xyz="0.05 ${lr * 0.01} -0.02" rpy="0 0 -1.570796327" /> <!-- TODO: guessed y offset -->
         <geometry>
-          <mesh filename="/home/sander/src/boldbot/boldbot_description/meshes/nicefoot${side}.stl" scale="0.001 0.001 0.001"/>
+          <mesh filename="$(find boldbot_description)/meshes/nicefoot${side}.stl" scale="0.001 0.001 0.001"/>
         </geometry>
       </collision>

Commit message: Use runtime package resolution rather than compile time

File: boldbot_description/urdf/boldbot.urdf.xacro (robot description, xacro)
@@ -6,5 +6,5 @@
         <origin xyz="${xyz}" rpy="${rpy}" />
         <geometry>
-          <mesh filename="$(find boldbot_description)/meshes/mx28.stl" scale="0.001 0.001 0.001" />
+          <mesh filename="package://boldbot_description/meshes/mx28.stl" scale="0.001 0.001 0.001" />
         </geometry>
         <material name="DarkGrey">
@@ -15,5 +15,5 @@
         <origin xyz="${xyz}" rpy="${rpy}" />
         <geometry>
-          <mesh filename="$(find boldbot_description)/meshes/mx28.stl" scale="0.001 0.001 0.001" />
+          <mesh filename="package://boldbot_description/meshes/mx28.stl" scale="0.001 0.001 0.001" />
         </geometry>
       </collision>
@@ -175,5 +175,5 @@
         <origin xyz="0.055 ${lr * 0.02} -0.02" rpy="${lr * 1.570796327} 0 0" />
         <geometry>
-          <mesh filename="$(find boldbot_description)/meshes/armcover.stl" scale="0.001 0.001 0.001"/>
+          <mesh filename="package://boldbot_description/meshes/armcover.stl" scale="0.001 0.001 0.001"/>
         </geometry>
       </visual>
@@ -181,5 +181,5 @@
         <origin xyz="0.055 ${lr * 0.02} -0.02" rpy="${lr * 1.570796327} 0 0" />
         <geometry>
-          <mesh filename="$(find boldbot_description)/meshes/armcover.stl" scale="0.001 0.001 0.001"/>
+          <mesh filename="package://boldbot_description/meshes/armcover.stl" scale="0.001 0.001 0.001"/>
         </geometry>
       </collision>
@@ -245,5 +245,5 @@
         <origin xyz="0 0 0" rpy="0 1.570796327 0" />
         <geometry>
-          <mesh filename="$(find boldbot_description)/meshes/thigh.stl" scale="0.001 0.001 0.001"/>
+          <mesh filename="package://boldbot_description/meshes/thigh.stl" scale="0.001 0.001 0.001"/>
         </geometry>
       </visual>
@@ -251,5 +251,5 @@
         <origin xyz="0 0 0" rpy="0 1.570796327 0" />
         <geometry>
-          <mesh filename="$(find boldbot_description)/meshes/thigh.stl" scale="0.001 0.001 0.001"/>
+          <mesh filename="package://boldbot_description/meshes/thigh.stl" scale="0.001 0.001 0.001"/>
         </geometry>
       </collision>
@@ -281,5 +281,5 @@
         <origin xyz="0.0175 0 -0.019" rpy="3.141592654 1.570796327 0" />
         <geometry>
-          <mesh filename="$(find boldbot_description)/meshes/shin.stl" scale="0.001 0.001 0.001"/>
+          <mesh filename="package://boldbot_description/meshes/shin.stl" scale="0.001 0.001 0.001"/>
         </geometry>
       </visual>
@@ -287,5 +287,5 @@
         <origin xyz="0.0175 0 -0.019" rpy="3.141592654 1.570796327 0" />
         <geometry>
-          <mesh filename="$(find boldbot_description)/meshes/shin.stl" scale="0.001 0.001 0.001"/>
+          <mesh filename="package://boldbot_description/meshes/shin.stl" scale="0.001 0.001 0.001"/>
         </geometry>
       </collision>
@@ -325,5 +325,5 @@
         <origin xyz="0.05 ${lr * 0.01} -0.02" rpy="0 0 -1.570796327" /> <!-- TODO: guessed y offset -->
         <geometry>
-          <mesh filename="$(find boldbot_description)/meshes/nicefoot${side}.stl" scale="0.001 0.001 0.001"/>
+          <mesh filename="package://boldbot_description/meshes/nicefoot${side}.stl" scale="0.001 0.001 0.001"/>
         </geometry>
       </visual>
@@ -331,5 +331,5 @@
         <origin xyz="0.05 ${lr * 0.01} -0.02" rpy="0 0 -1.570796327" /> <!-- TODO: guessed y offset -->
         <geometry>
-          <mesh filename="$(find boldbot_description)/meshes/nicefoot${side}.stl" scale="0.001 0.001 0.001"/>
+          <mesh filename="package://boldbot_description/meshes/nicefoot${side}.stl" scale="0.001 0.001 0.001"/>
         </geometry>
       </collision>

Commit message: Fix role -> roll

File: boldbot_description/urdf/boldbot.urdf.xacro (robot description, xacro)
@@ -308,12 +308,12 @@
     </joint>
     <xacro:mx28 name="mx28-ankle-pitch-${side}" xyz="0 0 0" rpy="1.570796327 -1.570796327 0"/>
-    <joint name="mx28-ankle-pitch-mx28-ankle-role-${side}" type="fixed">
+    <joint name="mx28-ankle-pitch-mx28-ankle-roll-${side}" type="fixed">
       <parent link="mx28-ankle-pitch-${side}" />
-      <child link="mx28-ankle-role-${side}" />
+      <child link="mx28-ankle-roll-${side}" />
       <origin xyz="-0.05 0 0" rpy="0 0 0" />
     </joint>
-    <xacro:mx28 name="mx28-ankle-role-${side}" xyz="0 0 0" rpy="3.141592654 -1.570796327 0"/>
-    <joint name="mx28-ankle-role-foot-${side}" type="continuous">
-      <parent link="mx28-ankle-role-${side}" />
+    <xacro:mx28 name="mx28-ankle-roll-${side}" xyz="0 0 0" rpy="3.141592654 -1.570796327 0"/>
+    <joint name="mx28-ankle-roll-foot-${side}" type="continuous">
+      <parent link="mx28-ankle-roll-${side}" />
       <child link="foot-${side}" />
       <origin xyz="0 0 0" rpy="0 0 0" />

Commit message: Find movable joints

File: boldbot_description/urdf/boldbot.urdf.xacro (robot description, xacro)
@@ -234,5 +234,5 @@
     </joint>
     <xacro:mx28 name="mx28-hip-pitch-${side}" xyz="0 0 0" rpy="1.570796327 1.570796327 0"/>
-    <joint name="mx28-hip-pitch-upper-leg-${side}" type="continuous">
+    <joint name="hip-pitch-${side}" type="continuous">
       <parent link="mx28-hip-pitch-${side}" />
       <child link="upper-leg-${side}" />
@@ -270,5 +270,5 @@
     </joint>
     <xacro:mx28 name="mx28-knee-${side}" xyz="0 0 0" rpy="1.570796327 -1.570796327 0"/>
-    <joint name="mx28-knee-lower-leg-${side}" type="continuous">
+    <joint name="knee-${side}" type="continuous">
       <parent link="mx28-knee-${side}" />
       <child link="lower-leg-${side}" />
@@ -300,5 +300,5 @@
       <selfCollide>true</selfCollide>
     </gazebo>
-    <joint name="lower-leg-mx28-ankle-pitch-${side}" type="continuous">
+    <joint name="ankle-pitch-${side}" type="continuous">
       <parent link="lower-leg-${side}" />
       <child link="mx28-ankle-pitch-${side}" />
@@ -314,5 +314,5 @@
     </joint>
     <xacro:mx28 name="mx28-ankle-roll-${side}" xyz="0 0 0" rpy="3.141592654 -1.570796327 0"/>
-    <joint name="mx28-ankle-roll-foot-${side}" type="continuous">
+    <joint name="ankle-roll-${side}" type="continuous">
       <parent link="mx28-ankle-roll-${side}" />
       <child link="foot-${side}" />

Commit message: Add camera sensor

File: boldbot_description/urdf/boldbot.urdf.xacro (robot description, xacro)
@@ -4,22 +4,22 @@
     <link name="${name}">
       <visual>
-        <origin xyz="${xyz}" rpy="${rpy}" />
-        <geometry>
-          <mesh filename="package://boldbot_description/meshes/mx28.stl" scale="0.001 0.001 0.001" />
-        </geometry>
-        <material name="DarkGrey">
-          <color rgba="0.20 0.20 0.20 1.0"/>
-        </material>
-      </visual>
-      <collision>
-        <origin xyz="${xyz}" rpy="${rpy}" />
-        <geometry>
-          <mesh filename="package://boldbot_description/meshes/mx28.stl" scale="0.001 0.001 0.001" />
-        </geometry>
-      </collision>
-      <inertial>
-        <origin xyz="${xyz}" rpy="${rpy}" />
-        <mass value="0.072"/>
-        <inertia ixx="0.00002292366"  ixy="0.0"  ixz="0.0" iyy="0.00001516566" iyz="0.0" izz="0.00002296632" />
+	<origin xyz="${xyz}" rpy="${rpy}" />
+	<geometry>
+	  <mesh filename="package://boldbot_description/meshes/mx28.stl" scale="0.001 0.001 0.001" />
+	</geometry>
+	<material name="DarkGrey">
+	  <color rgba="0.20 0.20 0.20 1.0"/>
+	</material>
+      </visual>
+      <collision>
+	<origin xyz="${xyz}" rpy="${rpy}" />
+	<geometry>
+	  <mesh filename="package://boldbot_description/meshes/mx28.stl" scale="0.001 0.001 0.001" />
+	</geometry>
+      </collision>
+      <inertial>
+	<origin xyz="${xyz}" rpy="${rpy}" />
+	<mass value="0.072"/>
+	<inertia ixx="0.00002292366"  ixy="0.0"  ixz="0.0" iyy="0.00001516566" iyz="0.0" izz="0.00002296632" />
       </inertial>
     </link>
@@ -40,5 +40,5 @@
       <origin rpy="0 0 0" xyz="0 0 0" />
       <geometry>
-        <box size="0.1 0.109 0.045"/>
+	<box size="0.1 0.109 0.045"/>
       </geometry>
     </visual>
@@ -46,5 +46,5 @@
       <origin rpy="0 0 0" xyz="0 0 0" />
       <geometry>
-        <box size="0.1 0.109 0.045"/>
+	<box size="0.1 0.109 0.045"/>
       </geometry>
     </collision>
@@ -76,5 +76,5 @@
       <origin rpy="0 0 0" xyz="0 0 0.03" />
       <geometry>
-        <box size="0.01 0.01 0.01"/>
+	<box size="0.01 0.01 0.01"/>
       </geometry>
     </visual>
@@ -102,5 +102,5 @@
       <origin rpy="0 0 0" xyz="0 0 0"/>
       <geometry>
-        <box size="0.05 0.1 0.04" />
+	<box size="0.05 0.1 0.04" />
       </geometry>
     </visual>
@@ -108,5 +108,5 @@
       <origin rpy="0 0 0" xyz="0 0 0"/>
       <geometry>
-        <box size="0.05 0.1 0.04" />
+	<box size="0.05 0.1 0.04" />
       </geometry>
     </collision>
@@ -139,13 +139,13 @@
     <link name="shoulder-${side}">
       <visual>
-        <origin rpy="0 0 0" xyz="0 ${lr * 0.021} -0.008" />
-        <geometry>
-          <box size="0.01 0.01 0.01"/>
-        </geometry>
-      </visual>
-      <inertial>
-        <origin xyz="0 0 0" />
-        <mass value="0.1"/>
-        <inertia ixx="1e-4"  ixy="0.0"  ixz="0.0" iyy="1e-4" iyz="0.0" izz="1e-4" />
+	<origin rpy="0 0 0" xyz="0 ${lr * 0.021} -0.008" />
+	<geometry>
+	  <box size="0.01 0.01 0.01"/>
+	</geometry>
+      </visual>
+      <inertial>
+	<origin xyz="0 0 0" />
+	<mass value="0.1"/>
+	<inertia ixx="1e-4"  ixy="0.0"  ixz="0.0" iyy="1e-4" iyz="0.0" izz="1e-4" />
       </inertial>
     </link>
@@ -173,19 +173,19 @@
     <link name="lower-arm-${side}">
       <visual>
-        <origin xyz="0.055 ${lr * 0.02} -0.02" rpy="${lr * 1.570796327} 0 0" />
-        <geometry>
-          <mesh filename="package://boldbot_description/meshes/armcover.stl" scale="0.001 0.001 0.001"/>
-        </geometry>
-      </visual>
-      <collision>
-        <origin xyz="0.055 ${lr * 0.02} -0.02" rpy="${lr * 1.570796327} 0 0" />
-        <geometry>
-          <mesh filename="package://boldbot_description/meshes/armcover.stl" scale="0.001 0.001 0.001"/>
-        </geometry>
-      </collision>
-      <inertial>
-        <origin xyz="0 0 0" />
-        <mass value="0.1"/>
-        <inertia ixx="1e-3"  ixy="0.0"  ixz="0.0" iyy="1e-3" iyz="0.0" izz="1e-3" />
+	<origin xyz="0.055 ${lr * 0.02} -0.02" rpy="${lr * 1.570796327} 0 0" />
+	<geometry>
+	  <mesh filename="package://boldbot_description/meshes/armcover.stl" scale="0.001 0.001 0.001"/>
+	</geometry>
+      </visual>
+      <collision>
+	<origin xyz="0.055 ${lr * 0.02} -0.02" rpy="${lr * 1.570796327} 0 0" />
+	<geometry>
+	  <mesh filename="package://boldbot_description/meshes/armcover.stl" scale="0.001 0.001 0.001"/>
+	</geometry>
+      </collision>
+      <inertial>
+	<origin xyz="0 0 0" />
+	<mass value="0.1"/>
+	<inertia ixx="1e-3"  ixy="0.0"  ixz="0.0" iyy="1e-3" iyz="0.0" izz="1e-3" />
       </inertial>
     </link>
@@ -215,7 +215,7 @@
     <link name="hip-bracket-${side}">
       <inertial>
-        <origin xyz="0 0 0" />
-        <mass value=".1"/>
-        <inertia ixx="1e-4"  ixy="0.0"  ixz="0.0" iyy="1e-4" iyz="0.0" izz="1e-4" />
+	<origin xyz="0 0 0" />
+	<mass value=".1"/>
+	<inertia ixx="1e-4"  ixy="0.0"  ixz="0.0" iyy="1e-4" iyz="0.0" izz="1e-4" />
       </inertial>
     </link>
@@ -243,19 +243,19 @@
     <link name="upper-leg-${side}">
       <visual>
-        <origin xyz="0 0 0" rpy="0 1.570796327 0" />
-        <geometry>
-          <mesh filename="package://boldbot_description/meshes/thigh.stl" scale="0.001 0.001 0.001"/>
-        </geometry>
-      </visual>
-      <collision>
-        <origin xyz="0 0 0" rpy="0 1.570796327 0" />
-        <geometry>
-          <mesh filename="package://boldbot_description/meshes/thigh.stl" scale="0.001 0.001 0.001"/>
-        </geometry>
-      </collision>
-      <inertial>
-        <origin xyz="0 0 0" />
-        <mass value="0.1"/>
-        <inertia ixx="1e-3"  ixy="0.0"  ixz="0.0" iyy="1e-3" iyz="0.0" izz="1e-3" />
+	<origin xyz="0 0 0" rpy="0 1.570796327 0" />
+	<geometry>
+	  <mesh filename="package://boldbot_description/meshes/thigh.stl" scale="0.001 0.001 0.001"/>
+	</geometry>
+      </visual>
+      <collision>
+	<origin xyz="0 0 0" rpy="0 1.570796327 0" />
+	<geometry>
+	  <mesh filename="package://boldbot_description/meshes/thigh.stl" scale="0.001 0.001 0.001"/>
+	</geometry>
+      </collision>
+      <inertial>
+	<origin xyz="0 0 0" />
+	<mass value="0.1"/>
+	<inertia ixx="1e-3"  ixy="0.0"  ixz="0.0" iyy="1e-3" iyz="0.0" izz="1e-3" />
       </inertial>
     </link>
@@ -279,19 +279,19 @@
     <link name="lower-leg-${side}">
       <visual>
-        <origin xyz="0.0175 0 -0.019" rpy="3.141592654 1.570796327 0" />
-        <geometry>
-          <mesh filename="package://boldbot_description/meshes/shin.stl" scale="0.001 0.001 0.001"/>
-        </geometry>
-      </visual>
-      <collision>
-        <origin xyz="0.0175 0 -0.019" rpy="3.141592654 1.570796327 0" />
-        <geometry>
-          <mesh filename="package://boldbot_description/meshes/shin.stl" scale="0.001 0.001 0.001"/>
-        </geometry>
-      </collision>
-      <inertial>
-        <origin xyz="0 0 0" />
-        <mass value="0.1"/>
-        <inertia ixx="1e-3"  ixy="0.0"  ixz="0.0" iyy="1e-3" iyz="0.0" izz="1e-3" />
+	<origin xyz="0.0175 0 -0.019" rpy="3.141592654 1.570796327 0" />
+	<geometry>
+	  <mesh filename="package://boldbot_description/meshes/shin.stl" scale="0.001 0.001 0.001"/>
+	</geometry>
+      </visual>
+      <collision>
+	<origin xyz="0.0175 0 -0.019" rpy="3.141592654 1.570796327 0" />
+	<geometry>
+	  <mesh filename="package://boldbot_description/meshes/shin.stl" scale="0.001 0.001 0.001"/>
+	</geometry>
+      </collision>
+      <inertial>
+	<origin xyz="0 0 0" />
+	<mass value="0.1"/>
+	<inertia ixx="1e-3"  ixy="0.0"  ixz="0.0" iyy="1e-3" iyz="0.0" izz="1e-3" />
       </inertial>
     </link>
@@ -323,19 +323,19 @@
     <link name="foot-${side}">
       <visual>
-        <origin xyz="0.05 ${lr * 0.01} -0.02" rpy="0 0 -1.570796327" /> <!-- TODO: guessed y offset -->
-        <geometry>
-          <mesh filename="package://boldbot_description/meshes/nicefoot${side}.stl" scale="0.001 0.001 0.001"/>
-        </geometry>
-      </visual>
-      <collision>
-        <origin xyz="0.05 ${lr * 0.01} -0.02" rpy="0 0 -1.570796327" /> <!-- TODO: guessed y offset -->
-        <geometry>
-          <mesh filename="package://boldbot_description/meshes/nicefoot${side}.stl" scale="0.001 0.001 0.001"/>
-        </geometry>
-      </collision>
-      <inertial>
-        <origin xyz="0 0 0" />
-        <mass value="0.1"/>
-        <inertia ixx="1e-3"  ixy="0.0"  ixz="0.0" iyy="1e-3" iyz="0.0" izz="1e-3" />
+	<origin xyz="0.05 ${lr * 0.01} -0.02" rpy="0 0 -1.570796327" /> <!-- TODO: guessed y offset -->
+	<geometry>
+	  <mesh filename="package://boldbot_description/meshes/nicefoot${side}.stl" scale="0.001 0.001 0.001"/>
+	</geometry>
+      </visual>
+      <collision>
+	<origin xyz="0.05 ${lr * 0.01} -0.02" rpy="0 0 -1.570796327" /> <!-- TODO: guessed y offset -->
+	<geometry>
+	  <mesh filename="package://boldbot_description/meshes/nicefoot${side}.stl" scale="0.001 0.001 0.001"/>
+	</geometry>
+      </collision>
+      <inertial>
+	<origin xyz="0 0 0" />
+	<mass value="0.1"/>
+	<inertia ixx="1e-3"  ixy="0.0"  ixz="0.0" iyy="1e-3" iyz="0.0" izz="1e-3" />
       </inertial>
     </link>
@@ -351,3 +351,36 @@
     </plugin>
   </gazebo>
+  <gazebo reference="head">
+    <sensor name='camera' type='camera'>
+      <pose>0 0 0 0 0 0</pose>
+      <camera name='__default__'>
+	<horizontal_fov>1.012300</horizontal_fov>
+	<image>
+	  <width>640</width>
+	  <height>480</height>
+	</image>
+	<clip>
+	  <near>0.001000</near>
+	  <far>100.000000</far>
+	</clip>
+      </camera>
+      <always_on>1</always_on>
+      <update_rate>30.000000</update_rate>
+      <visualize>1</visualize>
+      <plugin name="camera_controller" filename="libgazebo_ros_camera.so">
+	<alwaysOn>true</alwaysOn>
+	<updateRate>30</updateRate>
+	<cameraName>darwin/camera</cameraName>
+	<imageTopicName>image_raw</imageTopicName>
+	<cameraInfoTopicName>camera_info</cameraInfoTopicName>
+	<frameName>camera_link</frameName>
+	<hackBaseline>0.07</hackBaseline>
+	<distortionK1>0.0</distortionK1>
+	<distortionK2>0.0</distortionK2>
+	<distortionK3>0.0</distortionK3>
+	<distortionT1>0.0</distortionT1>
+	<distortionT2>0.0</distortionT2>
+      </plugin>
+    </sensor>
+  </gazebo>
 </robot>

Commit message: Make all joints revolute and flip left and right properly

File: boldbot_description/urdf/boldbot.urdf.xacro (robot description, xacro)
@@ -206,5 +206,5 @@
     </joint>
     <xacro:mx28 name="mx28-hip-yaw-${side}" xyz="0 0 0" rpy="${lr * 3.141592654} 0 3.141592654"/>
-    <joint name="hip-yaw-${side}" type="continuous">
+    <joint name="hip-yaw-${side}" type="revolute">
       <parent link="mx28-hip-yaw-${side}" />
       <child link="hip-bracket-${side}" />
@@ -220,5 +220,5 @@
       </inertial>
     </link>
-    <joint name="hip-roll-${side}" type="continuous">
+    <joint name="hip-roll-${side}" type="revolute">
       <parent link="hip-bracket-${side}" />
       <child link="mx28-hip-roll-${side}" />
@@ -234,9 +234,9 @@
     </joint>
     <xacro:mx28 name="mx28-hip-pitch-${side}" xyz="0 0 0" rpy="1.570796327 1.570796327 0"/>
-    <joint name="hip-pitch-${side}" type="continuous">
+    <joint name="hip-pitch-${side}" type="revolute">
       <parent link="mx28-hip-pitch-${side}" />
       <child link="upper-leg-${side}" />
       <origin xyz="0 0 0" rpy="0 0 0" />
-      <axis xyz="0 -1 0" />
+      <axis xyz="0 ${lr * -1} 0" />
       <limit effort="2.8" velocity="5.6548668" lower="-2.6179939" upper="2.6179939" />
     </joint>
@@ -270,9 +270,9 @@
     </joint>
     <xacro:mx28 name="mx28-knee-${side}" xyz="0 0 0" rpy="1.570796327 -1.570796327 0"/>
-    <joint name="knee-${side}" type="continuous">
+    <joint name="knee-${side}" type="revolute">
       <parent link="mx28-knee-${side}" />
       <child link="lower-leg-${side}" />
       <origin xyz="0 0 0" rpy="0 0 0" />
-      <axis xyz="0 -1 0" />
+      <axis xyz="0 ${lr * -1} 0" />
       <limit effort="2.8" velocity="5.6548668" lower="-2.6179939" upper="2.6179939" />
     </joint>
@@ -300,9 +300,9 @@
       <selfCollide>true</selfCollide>
     </gazebo>
-    <joint name="ankle-pitch-${side}" type="continuous">
+    <joint name="ankle-pitch-${side}" type="revolute">
       <parent link="lower-leg-${side}" />
       <child link="mx28-ankle-pitch-${side}" />
       <origin xyz="0 0 -0.143" rpy="0 0 0" />
-      <axis xyz="0 -1 0" />
+      <axis xyz="0 ${lr * 1} 0" />
       <limit effort="2.8" velocity="5.6548668" lower="-2.6179939" upper="2.6179939" />
     </joint>
@@ -314,5 +314,5 @@
     </joint>
     <xacro:mx28 name="mx28-ankle-roll-${side}" xyz="0 0 0" rpy="3.141592654 -1.570796327 0"/>
-    <joint name="ankle-roll-${side}" type="continuous">
+    <joint name="ankle-roll-${side}" type="revolute">
       <parent link="mx28-ankle-roll-${side}" />
       <child link="foot-${side}" />
