Commit message: Start calculating inertia automatically based on box model

File: boldbot_description/urdf/boldbot.urdf.xacro (robot description, xacro)
@@ -1,4 +1,13 @@
 <?xml version="1.0" ?>
 <robot name="boldbot" xmlns:xacro="http://www.ros.org/wiki/xacro">
+  <xacro:macro name="inertial_cuboid" params="mass x_length y_length z_length">
+    <inertial>
+      <mass value="${mass}" />
+      <origin xyz="0 0 0" />
+      <inertia ixx="${(1/12) * mass * (y_length*y_length + z_length*z_length)}" ixy="0.0" ixz="0.0"
+	       iyy="${(1/12) * mass * (x_length*x_length + z_length*z_length)}" iyz="0.0"
+	       izz="${(1/12) * mass * (x_length*x_length + y_length*y_length)}" />
+    </inertial>
+  </xacro:macro>
   <xacro:macro name="mx28" params="name xyz rpy">
     <link name="${name}">
@@ -18,9 +27,5 @@
 	</geometry>
       </collision>
-      <inertial>
-	<origin xyz="${xyz}" rpy="${rpy}" />
-	<mass value="0.072"/>
-	<inertia ixx="0.00002292366"  ixy="0.0"  ixz="0.0" iyy="0.00001516566" iyz="0.0" izz="0.00002296632" />
-      </inertial>
+      <xacro:inertial_cuboid mass="0.077" x_length="0.0506" y_length="0.0356" z_length="0.0355" />
     </link>
     <gazebo reference="${name}">
@@ -49,9 +54,5 @@
       </geometry>
     </collision>
-    <inertial>
-      <origin xyz="0 0 0" />
-      <mass value="0.1"/>
-      <inertia ixx="1e-3"  ixy="0.0"  ixz="0.0" iyy="1e-3" iyz="0.0" izz="1e-3" />
-    </inertial>
+    <xacro:inertial_cuboid mass="0.31" x_length="0.1" y_length="0.109" z_length="0.045"/>
   </link>
   <gazebo reference="torso">

Commit message: Add launch file and export/change some paths to make it work

File: boldbot_description/urdf/boldbot.urdf.xacro (robot description, xacro)
@@ -15,5 +15,5 @@
 	<origin xyz="${xyz}" rpy="${rpy}" />
 	<geometry>
-	  <mesh filename="package://boldbot_description/meshes/mx28.stl" scale="0.001 0.001 0.001" />
+	  <mesh filename="package://meshes/mx28.stl" scale="0.001 0.001 0.001" />
 	</geometry>
 	<material name="DarkGrey">
@@ -24,5 +24,5 @@
 	<origin xyz="${xyz}" rpy="${rpy}" />
 	<geometry>
-	  <mesh filename="package://boldbot_description/meshes/mx28.stl" scale="0.001 0.001 0.001" />
+	  <mesh filename="package://meshes/mx28.stl" scale="0.001 0.001 0.001" />
 	</geometry>
       </collision>
@@ -176,5 +176,5 @@
 	<origin xyz="0.055 ${lr * 0.02} -0.02" rpy="${lr * 1.570796327} 0 0" />
 	<geometry>
-	  <mesh filename="package://boldbot_description/meshes/armcover.stl" scale="0.001 0.001 0.001"/>
+	  <mesh filename="package://meshes/armcover.stl" scale="0.001 0.001 0.001"/>
 	</geometry>
       </visual>
@@ -182,5 +182,5 @@
 	<origin xyz="0.055 ${lr * 0.02} -0.02" rpy="${lr * 1.570796327} 0 0" />
 	<geometry>
-	  <mesh filename="package://boldbot_description/meshes/armcover.stl" scale="0.001 0.001 0.001"/>
+	  <mesh filename="package://meshes/armcover.stl" scale="0.001 0.001 0.001"/>
 	</geometry>
       </collision>
@@ -246,5 +246,5 @@
 	<origin xyz="0 0 0" rpy="0 1.570796327 0" />
 	<geometry>
-	  <mesh filename="package://boldbot_description/meshes/thigh.stl" scale="0.001 0.001 0.001"/>
+	  <mesh filename="package://meshes/thigh.stl" scale="0.001 0.001 0.001"/>
 	</geometry>
       </visual>
@@ -252,5 +252,5 @@
 	<origin xyz="0 0 0" rpy="0 1.570796327 0" />
 	<geometry>
-	  <mesh filename="package://boldbot_description/meshes/thigh.stl" scale="0.001 0.001 0.001"/>
+	  <mesh filename="package://meshes/thigh.stl" scale="0.001 0.001 0.001"/>
 	</geometry>
       </collision>
@@ -282,5 +282,5 @@
 	<origin xyz="0.0175 0 -0.019" rpy="3.141592654 1.570796327 0" />
 	<geometry>
-	  <mesh filename="package://boldbot_description/meshes/shin.stl" scale="0.001 0.001 0.001"/>
+	  <mesh filename="package://meshes/shin.stl" scale="0.001 0.001 0.001"/>
 	</geometry>
       </visual>
@@ -288,5 +288,5 @@
 	<origin xyz="0.0175 0 -0.019" rpy="3.141592654 1.570796327 0" />
 	<geometry>
-	  <mesh filename="package://boldbot_description/meshes/shin.stl" scale="0.001 0.001 0.001"/>
+	  <mesh filename="package://meshes/shin.stl" scale="0.001 0.001 0.001"/>
 	</geometry>
       </collision>
@@ -326,5 +326,5 @@
 	<origin xyz="0.05 ${lr * 0.01} -0.02" rpy="0 0 -1.570796327" /> <!-- TODO: guessed y offset -->
 	<geometry>
-	  <mesh filename="package://boldbot_description/meshes/nicefoot${side}.stl" scale="0.001 0.001 0.001"/>
+	  <mesh filename="package://meshes/nicefoot${side}.stl" scale="0.001 0.001 0.001"/>
 	</geometry>
       </visual>
@@ -332,5 +332,5 @@
 	<origin xyz="0.05 ${lr * 0.01} -0.02" rpy="0 0 -1.570796327" /> <!-- TODO: guessed y offset -->
 	<geometry>
-	  <mesh filename="package://boldbot_description/meshes/nicefoot${side}.stl" scale="0.001 0.001 0.001"/>
+	  <mesh filename="package://meshes/nicefoot${side}.stl" scale="0.001 0.001 0.001"/>
 	</geometry>
       </collision>

Commit message: Update locations & paths to make model work with both gazebo & rviz

File: boldbot_description/urdf/boldbot.urdf.xacro (robot description, xacro)
@@ -15,5 +15,5 @@
 	<origin xyz="${xyz}" rpy="${rpy}" />
 	<geometry>
-	  <mesh filename="package://meshes/mx28.stl" scale="0.001 0.001 0.001" />
+	  <mesh filename="package://boldbot_description/meshes/mx28b.stl" scale="0.001 0.001 0.001" />
 	</geometry>
 	<material name="DarkGrey">
@@ -24,5 +24,5 @@
 	<origin xyz="${xyz}" rpy="${rpy}" />
 	<geometry>
-	  <mesh filename="package://meshes/mx28.stl" scale="0.001 0.001 0.001" />
+	  <mesh filename="package://boldbot_description/meshes/mx28b.stl" scale="0.001 0.001 0.001" />
 	</geometry>
       </collision>
@@ -176,5 +176,5 @@
 	<origin xyz="0.055 ${lr * 0.02} -0.02" rpy="${lr * 1.570796327} 0 0" />
 	<geometry>
-	  <mesh filename="package://meshes/armcover.stl" scale="0.001 0.001 0.001"/>
+	  <mesh filename="package://boldbot_description/meshes/armcoverb.stl" scale="0.001 0.001 0.001"/>
 	</geometry>
       </visual>
@@ -182,5 +182,5 @@
 	<origin xyz="0.055 ${lr * 0.02} -0.02" rpy="${lr * 1.570796327} 0 0" />
 	<geometry>
-	  <mesh filename="package://meshes/armcover.stl" scale="0.001 0.001 0.001"/>
+	  <mesh filename="package://boldbot_description/meshes/armcoverb.stl" scale="0.001 0.001 0.001"/>
 	</geometry>
       </collision>
@@ -246,5 +246,5 @@
 	<origin xyz="0 0 0" rpy="0 1.570796327 0" />
 	<geometry>
-	  <mesh filename="package://meshes/thigh.stl" scale="0.001 0.001 0.001"/>
+	  <mesh filename="package://boldbot_description/meshes/thighb.stl" scale="0.001 0.001 0.001"/>
 	</geometry>
       </visual>
@@ -252,5 +252,5 @@
 	<origin xyz="0 0 0" rpy="0 1.570796327 0" />
 	<geometry>
-	  <mesh filename="package://meshes/thigh.stl" scale="0.001 0.001 0.001"/>
+	  <mesh filename="package://boldbot_description/meshes/thighb.stl" scale="0.001 0.001 0.001"/>
 	</geometry>
       </collision>
@@ -282,5 +282,5 @@
 	<origin xyz="0.0175 0 -0.019" rpy="3.141592654 1.570796327 0" />
 	<geometry>
-	  <mesh filename="package://meshes/shin.stl" scale="0.001 0.001 0.001"/>
+	  <mesh filename="package://boldbot_description/meshes/shinb.stl" scale="0.001 0.001 0.001"/>
 	</geometry>
       </visual>
@@ -288,5 +288,5 @@
 	<origin xyz="0.0175 0 -0.019" rpy="3.141592654 1.570796327 0" />
 	<geometry>
-	  <mesh filename="package://meshes/shin.stl" scale="0.001 0.001 0.001"/>
+	  <mesh filename="package://boldbot_description/meshes/shinb.stl" scale="0.001 0.001 0.001"/>
 	</geometry>
       </collision>
@@ -326,5 +326,5 @@
 	<origin xyz="0.05 ${lr * 0.01} -0.02" rpy="0 0 -1.570796327" /> <!-- TODO: guessed y offset -->
 	<geometry>
-	  <mesh filename="package://meshes/nicefoot${side}.stl" scale="0.001 0.001 0.001"/>
+	  <mesh filename="package://boldbot_description/meshes/nicefoot${side}b.stl" scale="0.001 0.001 0.001"/>
 	</geometry>
       </visual>
@@ -332,5 +332,5 @@
 	<origin xyz="0.05 ${lr * 0.01} -0.02" rpy="0 0 -1.570796327" /> <!-- TODO: guessed y offset -->
 	<geometry>
-	  <mesh filename="package://meshes/nicefoot${side}.stl" scale="0.001 0.001 0.001"/>
+	  <mesh filename="package://boldbot_description/meshes/nicefoot${side}b.stl" scale="0.001 0.001 0.001"/>
 	</geometry>
       </collision>

Commit message: Helper macros to test inertia sizes in Gazebo

File: boldbot_description/urdf/boldbot.urdf.xacro (robot description, xacro)
@@ -2,12 +2,24 @@
 <robot name="boldbot" xmlns:xacro="http://www.ros.org/wiki/xacro">
   <xacro:macro name="inertial_cuboid" params="mass x_length y_length z_length">
+  <xacro:macro name="xmass" params="value"><mass value="${value}" /></xacro:macro>
+  <!-- <xacro:macro name="xmass" params="value"><mass value="1" /></xacro:macro> -->
+  <xacro:macro name="inertial_cuboid" params="mass xyz x_length y_length z_length">
     <inertial>
-      <mass value="${mass}" />
-      <origin xyz="0 0 0" />
-      <inertia ixx="${(1/12) * mass * (y_length*y_length + z_length*z_length)}" ixy="0.0" ixz="0.0"
-	       iyy="${(1/12) * mass * (x_length*x_length + z_length*z_length)}" iyz="0.0"
-	       izz="${(1/12) * mass * (x_length*x_length + y_length*y_length)}" />
+      <xacro:xmass value="${mass}" />
+      <origin xyz="${xyz}" />
+      <inertia ixx="${mass * (y_length*y_length + z_length*z_length) / 12}" ixy="0.0" ixz="0.0"
+               iyy="${mass * (x_length*x_length + z_length*z_length) / 12}" iyz="0.0"
+               izz="${mass * (x_length*x_length + y_length*y_length) / 12}" />
     </inertial>
   </xacro:macro>
+  <!-- <xacro:macro name="inertial_cuboid" params="mass xyz x_length y_length z_length"> -->
+  <!--   <inertial> -->
+  <!--     <xacro:xmass value="1" /> -->
+  <!--     <origin xyz="${xyz}" /> -->
+  <!--     <inertia ixx="${1 * (y_length*y_length + z_length*z_length) / 12}" ixy="0.0" ixz="0.0" -->
+  <!--              iyy="${1 * (x_length*x_length + z_length*z_length) / 12}" iyz="0.0" -->
+  <!--              izz="${1 * (x_length*x_length + y_length*y_length) / 12}" /> -->
+  <!--   </inertial> -->
+  <!-- </xacro:macro> -->
   <xacro:macro name="mx28" params="name xyz rpy">
     <link name="${name}">

Commit message: Define properties for densities of printed pieces

File: boldbot_description/urdf/boldbot.urdf.xacro (robot description, xacro)
@@ -1,5 +1,8 @@
 <?xml version="1.0" ?>
 <robot name="boldbot" xmlns:xacro="http://www.ros.org/wiki/xacro">
-  <xacro:macro name="inertial_cuboid" params="mass x_length y_length z_length">
+  <!-- PLA: 1.24 g/cm^3 -->
+  <xacro:property name="filament_density_full" value="1240" />
+  <xacro:property name="infill" value=".5" />
+  <xacro:property name="filament_density" value="${filament_density_full * infill}" />
   <xacro:macro name="xmass" params="value"><mass value="${value}" /></xacro:macro>
   <!-- <xacro:macro name="xmass" params="value"><mass value="1" /></xacro:macro> -->

Commit message: Whitespace cleanup

File: boldbot_description/urdf/boldbot.urdf.xacro (robot description, xacro)
@@ -28,17 +28,17 @@
     <link name="${name}">
       <visual>
-	<origin xyz="${xyz}" rpy="${rpy}" />
-	<geometry>
-	  <mesh filename="package://boldbot_description/meshes/mx28b.stl" scale="0.001 0.001 0.001" />
-	</geometry>
-	<material name="DarkGrey">
-	  <color rgba="0.20 0.20 0.20 1.0"/>
-	</material>
+        <origin xyz="${xyz}" rpy="${rpy}" />
+        <geometry>
+          <mesh filename="package://boldbot_description/meshes/mx28b.stl" scale="0.001 0.001 0.001" />
+        </geometry>
+        <material name="DarkGrey">
+          <color rgba="0.20 0.20 0.20 1.0"/>
+        </material>
       </visual>
       <collision>
-	<origin xyz="${xyz}" rpy="${rpy}" />
-	<geometry>
-	  <mesh filename="package://boldbot_description/meshes/mx28b.stl" scale="0.001 0.001 0.001" />
-	</geometry>
+        <origin xyz="${xyz}" rpy="${rpy}" />
+        <geometry>
+          <mesh filename="package://boldbot_description/meshes/mx28b.stl" scale="0.001 0.001 0.001" />
+        </geometry>
       </collision>
       <xacro:inertial_cuboid mass="0.077" x_length="0.0506" y_length="0.0356" z_length="0.0355" />
@@ -60,5 +60,5 @@
       <origin rpy="0 0 0" xyz="0 0 0" />
       <geometry>
-	<box size="0.1 0.109 0.045"/>
+        <box size="0.1 0.109 0.045"/>
       </geometry>
     </visual>
@@ -66,5 +66,5 @@
       <origin rpy="0 0 0" xyz="0 0 0" />
       <geometry>
-	<box size="0.1 0.109 0.045"/>
+        <box size="0.1 0.109 0.045"/>
       </geometry>
     </collision>
@@ -92,5 +92,5 @@
       <origin rpy="0 0 0" xyz="0 0 0.03" />
       <geometry>
-	<box size="0.01 0.01 0.01"/>
+        <box size="0.01 0.01 0.01"/>
       </geometry>
     </visual>
@@ -118,5 +118,5 @@
       <origin rpy="0 0 0" xyz="0 0 0"/>
       <geometry>
-	<box size="0.05 0.1 0.04" />
+        <box size="0.05 0.1 0.04" />
       </geometry>
     </visual>
@@ -124,5 +124,5 @@
       <origin rpy="0 0 0" xyz="0 0 0"/>
       <geometry>
-	<box size="0.05 0.1 0.04" />
+        <box size="0.05 0.1 0.04" />
       </geometry>
     </collision>
@@ -155,13 +155,13 @@
     <link name="shoulder-${side}">
       <visual>
-	<origin rpy="0 0 0" xyz="0 ${lr * 0.021} -0.008" />
-	<geometry>
-	  <box size="0.01 0.01 0.01"/>
-	</geometry>
-      </visual>
-      <inertial>
-	<origin xyz="0 0 0" />
-	<mass value="0.1"/>
-	<inertia ixx="1e-4"  ixy="0.0"  ixz="0.0" iyy="1e-4" iyz="0.0" izz="1e-4" />
+        <origin rpy="0 0 0" xyz="0 ${lr * 0.021} -0.008" />
+        <geometry>
+          <box size="0.01 0.01 0.01"/>
+        </geometry>
+      </visual>
+      <inertial>
+        <origin xyz="0 0 0" />
+        <xacro:xmass value="0.1"/>
+        <inertia ixx="1e-4"  ixy="0.0"  ixz="0.0" iyy="1e-4" iyz="0.0" izz="1e-4" />
       </inertial>
     </link>
@@ -189,19 +189,19 @@
     <link name="lower-arm-${side}">
       <visual>
-	<origin xyz="0.055 ${lr * 0.02} -0.02" rpy="${lr * 1.570796327} 0 0" />
-	<geometry>
-	  <mesh filename="package://boldbot_description/meshes/armcoverb.stl" scale="0.001 0.001 0.001"/>
-	</geometry>
+        <origin xyz="0.055 ${lr * 0.02} -0.02" rpy="${lr * 1.570796327} 0 0" />
+        <geometry>
+          <mesh filename="package://boldbot_description/meshes/armcoverb.stl" scale="0.001 0.001 0.001"/>
+        </geometry>
       </visual>
       <collision>
-	<origin xyz="0.055 ${lr * 0.02} -0.02" rpy="${lr * 1.570796327} 0 0" />
-	<geometry>
-	  <mesh filename="package://boldbot_description/meshes/armcoverb.stl" scale="0.001 0.001 0.001"/>
-	</geometry>
+        <origin xyz="0.055 ${lr * 0.02} -0.02" rpy="${lr * 1.570796327} 0 0" />
+        <geometry>
+          <mesh filename="package://boldbot_description/meshes/armcoverb.stl" scale="0.001 0.001 0.001"/>
+        </geometry>
       </collision>
       <inertial>
-	<origin xyz="0 0 0" />
-	<mass value="0.1"/>
-	<inertia ixx="1e-3"  ixy="0.0"  ixz="0.0" iyy="1e-3" iyz="0.0" izz="1e-3" />
+        <origin xyz="0 0 0" />
+        <xacro:xmass value="0.1"/>
+        <inertia ixx="1e-3"  ixy="0.0"  ixz="0.0" iyy="1e-3" iyz="0.0" izz="1e-3" />
       </inertial>
     </link>
@@ -213,5 +213,5 @@
   <xacro:arm side="l"/>
   <xacro:arm side="r"/>
-  <!-- Left Leg -->
+  <!-- Legs -->
   <xacro:macro name="leg" params="side">
     <xacro:property name="lr" value="${1 if side == 'l' else -1}"/>
@@ -231,7 +231,7 @@
     <link name="hip-bracket-${side}">
       <inertial>
-	<origin xyz="0 0 0" />
-	<mass value=".1"/>
-	<inertia ixx="1e-4"  ixy="0.0"  ixz="0.0" iyy="1e-4" iyz="0.0" izz="1e-4" />
+        <origin xyz="0 0 0" />
+        <xacro:xmass value=".1"/>
+        <inertia ixx="1e-4"  ixy="0.0"  ixz="0.0" iyy="1e-4" iyz="0.0" izz="1e-4" />
       </inertial>
     </link>
@@ -259,19 +259,19 @@
     <link name="upper-leg-${side}">
       <visual>
-	<origin xyz="0 0 0" rpy="0 1.570796327 0" />
-	<geometry>
-	  <mesh filename="package://boldbot_description/meshes/thighb.stl" scale="0.001 0.001 0.001"/>
-	</geometry>
+        <origin xyz="0 0 0" rpy="0 1.570796327 0" />
+        <geometry>
+          <mesh filename="package://boldbot_description/meshes/thighb.stl" scale="0.001 0.001 0.001"/>
+        </geometry>
       </visual>
       <collision>
-	<origin xyz="0 0 0" rpy="0 1.570796327 0" />
-	<geometry>
-	  <mesh filename="package://boldbot_description/meshes/thighb.stl" scale="0.001 0.001 0.001"/>
-	</geometry>
+        <origin xyz="0 0 0" rpy="0 1.570796327 0" />
+        <geometry>
+          <mesh filename="package://boldbot_description/meshes/thighb.stl" scale="0.001 0.001 0.001"/>
+        </geometry>
       </collision>
       <inertial>
-	<origin xyz="0 0 0" />
-	<mass value="0.1"/>
-	<inertia ixx="1e-3"  ixy="0.0"  ixz="0.0" iyy="1e-3" iyz="0.0" izz="1e-3" />
+        <origin xyz="0 0 0" />
+        <xacro:xmass value="0.1"/>
+        <inertia ixx="1e-3"  ixy="0.0"  ixz="0.0" iyy="1e-3" iyz="0.0" izz="1e-3" />
       </inertial>
     </link>
@@ -295,14 +295,14 @@
     <link name="lower-leg-${side}">
       <visual>
-	<origin xyz="0.0175 0 -0.019" rpy="3.141592654 1.570796327 0" />
-	<geometry>
-	  <mesh filename="package://boldbot_description/meshes/shinb.stl" scale="0.001 0.001 0.001"/>
-	</geometry>
+        <origin xyz="0.0175 0 -0.019" rpy="3.141592654 1.570796327 0" />
+        <geometry>
+          <mesh filename="package://boldbot_description/meshes/shinb.stl" scale="0.001 0.001 0.001"/>
+        </geometry>
       </visual>
       <collision>
-	<origin xyz="0.0175 0 -0.019" rpy="3.141592654 1.570796327 0" />
-	<geometry>
-	  <mesh filename="package://boldbot_description/meshes/shinb.stl" scale="0.001 0.001 0.001"/>
-	</geometry>
+        <origin xyz="0.0175 0 -0.019" rpy="3.141592654 1.570796327 0" />
+        <geometry>
+          <mesh filename="package://boldbot_description/meshes/shinb.stl" scale="0.001 0.001 0.001"/>
+        </geometry>
       </collision>
       <inertial>
@@ -339,19 +339,19 @@
     <link name="foot-${side}">
       <visual>
-	<origin xyz="0.05 ${lr * 0.01} -0.02" rpy="0 0 -1.570796327" /> <!-- TODO: guessed y offset -->
-	<geometry>
-	  <mesh filename="package://boldbot_description/meshes/nicefoot${side}b.stl" scale="0.001 0.001 0.001"/>
-	</geometry>
+        <origin xyz="0.05 ${lr * 0.01} -0.02" rpy="0 0 -1.570796327" /> <!-- TODO: guessed y offset -->
+        <geometry>
+          <mesh filename="package://boldbot_description/meshes/nicefoot${side}b.stl" scale="0.001 0.001 0.001"/>
+        </geometry>
       </visual>
       <collision>
-	<origin xyz="0.05 ${lr * 0.01} -0.02" rpy="0 0 -1.570796327" /> <!-- TODO: guessed y offset -->
-	<geometry>
-	  <mesh filename="package://boldbot_description/meshes/nicefoot${side}b.stl" scale="0.001 0.001 0.001"/>
-	</geometry>
+        <origin xyz="0.05 ${lr * 0.01} -0.02" rpy="0 0 -1.570796327" /> <!-- TODO: guessed y offset -->
+        <geometry>
+          <mesh filename="package://boldbot_description/meshes/nicefoot${side}b.stl" scale="0.001 0.001 0.001"/>
+        </geometry>
       </collision>
       <inertial>
-	<origin xyz="0 0 0" />
-	<mass value="0.1"/>
-	<inertia ixx="1e-3"  ixy="0.0"  ixz="0.0" iyy="1e-3" iyz="0.0" izz="1e-3" />
+        <origin xyz="0 0 0" />
+        <xacro:xmass value="0.1"/>
+        <inertia ixx="1e-3"  ixy="0.0"  ixz="0.0" iyy="1e-3" iyz="0.0" izz="1e-3" />
       </inertial>
     </link>
@@ -371,13 +371,13 @@
       <pose>0 0 0 0 0 0</pose>
       <camera name='__default__'>
-	<horizontal_fov>1.012300</horizontal_fov>
-	<image>
-	  <width>640</width>
-	  <height>480</height>
-	</image>
-	<clip>
-	  <near>0.001000</near>
-	  <far>100.000000</far>
-	</clip>
+        <horizontal_fov>1.012300</horizontal_fov>
+        <image>
+          <width>640</width>
+          <height>480</height>
+        </image>
+        <clip>
+          <near>0.001000</near>
+          <far>100.000000</far>
+        </clip>
       </camera>
       <always_on>1</always_on>
@@ -385,16 +385,16 @@
       <visualize>true</visualize>
       <plugin name="camera_controller" filename="libgazebo_ros_camera.so">
-	<alwaysOn>true</alwaysOn>
-	<updateRate>30</updateRate>
-	<cameraName>darwin/camera</cameraName>
-	<imageTopicName>image_raw</imageTopicName>
-	<cameraInfoTopicName>camera_info</cameraInfoTopicName>
-	<frameName>camera_link</frameName>
-	<hackBaseline>0.07</hackBaseline>
-	<distortionK1>0.0</distortionK1>
-	<distortionK2>0.0</distortionK2>
-	<distortionK3>0.0</distortionK3>
-	<distortionT1>0.0</distortionT1>
-	<distortionT2>0.0</distortionT2>
+        <alwaysOn>true</alwaysOn>
+        <updateRate>30</updateRate>
+        <cameraName>darwin/camera</cameraName>
+        <imageTopicName>image_raw</imageTopicName>
+        <cameraInfoTopicName>camera_info</cameraInfoTopicName>
+        <frameName>camera_link</frameName>
+        <hackBaseline>0.07</hackBaseline>
+        <distortionK1>0.0</distortionK1>
+        <distortionK2>0.0</distortionK2>
+        <distortionK3>0.0</distortionK3>
+        <distortionT1>0.0</distortionT1>
+        <distortionT2>0.0</distortionT2>
       </plugin>
     </sensor>
@@ -408,9 +408,9 @@
       <topic>__default_topic__</topic>
       <plugin filename="libgazebo_ros_imu_sensor.so" name="imu_plugin">
-	<ros>
-	  <argument>~/out:=/imu/data_raw</argument>
-	</ros>
-	<bodyName>torso</bodyName>
-	<gaussianNoise>0.0</gaussianNoise>
+        <ros>
+          <argument>~/out:=/imu/data_raw</argument>
+        </ros>
+        <bodyName>torso</bodyName>
+        <gaussianNoise>0.0</gaussianNoise>
       </plugin>
       <pose>0 0 0 0 0 0</pose>

Commit message: Set head inertia from box sizes

File: boldbot_description/urdf/boldbot.urdf.xacro (robot description, xacro)
@@ -42,5 +42,5 @@
         </geometry>
       </collision>
-      <xacro:inertial_cuboid mass="0.077" x_length="0.0506" y_length="0.0356" z_length="0.0355" />
+      <xacro:inertial_cuboid mass="0.077" xyz="0 0 0" x_length="0.0506" y_length="0.0356" z_length="0.0355" />
     </link>
     <gazebo reference="${name}">
@@ -69,5 +69,5 @@
       </geometry>
     </collision>
-    <xacro:inertial_cuboid mass="0.31" x_length="0.1" y_length="0.109" z_length="0.045"/>
+    <xacro:inertial_cuboid mass="0.31" xyz="0 0 0" x_length="0.1" y_length="0.109" z_length="0.045"/>
   </link>
   <gazebo reference="torso">
@@ -97,5 +97,5 @@
     <inertial>
       <origin xyz="0 0 0" />
-      <mass value="1e-3"/>
+      <xacro:xmass value="1e-3"/>
       <inertia ixx="1e-4"  ixy="0.0"  ixz="0.0" iyy="1e-4" iyz="0.0" izz="1e-4" />
     </inertial>
@@ -127,9 +127,5 @@
       </geometry>
     </collision>
-    <inertial>
-      <origin xyz="0 0 0" />
-      <mass value=".2"/>
-      <inertia ixx="1e-3"  ixy="0.0"  ixz="0.0" iyy="1e-3" iyz="0.0" izz="1e-3" />
-    </inertial>
+    <xacro:inertial_cuboid mass="0.2" xyz="0 0 0" x_length="0.05" y_length="0.1" z_length="0.04" />
   </link>
   <gazebo reference="head">
