Commit message: Update inertias, MX28 is wrong

File: boldbot_description/urdf/boldbot.urdf.xacro (robot description, xacro)
@@ -5,10 +5,11 @@
   <xacro:property name="infill" value=".5" />
   <xacro:property name="filament_density" value="${filament_density_full * infill}" />
+  <xacro:property name="aluminium_density" value="2700" />
   <xacro:macro name="xmass" params="value"><mass value="${value}" /></xacro:macro>
   <!-- <xacro:macro name="xmass" params="value"><mass value="1" /></xacro:macro> -->
-  <xacro:macro name="inertial_cuboid" params="mass xyz x_length y_length z_length">
+  <xacro:macro name="inertial_cuboid" params="mass xyz rpy x_length y_length z_length">
     <inertial>
       <xacro:xmass value="${mass}" />
-      <origin xyz="${xyz}" />
+      <origin rpy="0 0 0" xyz="${xyz}"/>
       <inertia ixx="${mass * (y_length*y_length + z_length*z_length) / 12}" ixy="0.0" ixz="0.0"
                iyy="${mass * (x_length*x_length + z_length*z_length) / 12}" iyz="0.0"
@@ -25,8 +26,8 @@
   <!--   </inertial> -->
   <!-- </xacro:macro> -->
-  <xacro:macro name="mx28" params="name xyz rpy">
+  <xacro:macro name="mx28" params="name">
     <link name="${name}">
       <visual>
-        <origin xyz="${xyz}" rpy="${rpy}" />
+        <origin xyz="0 0 0" rpy="0 0 0" />
         <geometry>
           <mesh filename="package://boldbot_description/meshes/mx28b.stl" scale="0.001 0.001 0.001" />
@@ -37,10 +38,10 @@
       </visual>
       <collision>
-        <origin xyz="${xyz}" rpy="${rpy}" />
+        <origin xyz="0 0 0" rpy="0 0 0" />
         <geometry>
           <mesh filename="package://boldbot_description/meshes/mx28b.stl" scale="0.001 0.001 0.001" />
         </geometry>
       </collision>
-      <xacro:inertial_cuboid mass="0.077" xyz="0 0 0" x_length="0.0506" y_length="0.0356" z_length="0.0355" />
+      <xacro:inertial_cuboid mass="0.077" xyz="0.0105 0 0" rpy="0 0 0" x_length="0.0506" y_length="0.0356" z_length="0.0355" />
     </link>
     <gazebo reference="${name}">
@@ -69,5 +70,5 @@
       </geometry>
     </collision>
-    <xacro:inertial_cuboid mass="0.31" xyz="0 0 0" x_length="0.1" y_length="0.109" z_length="0.045"/>
+    <xacro:inertial_cuboid mass="0.31" xyz="0 0 0" rpy="0 0 0" x_length="0.1" y_length="0.109" z_length="0.045"/>
   </link>
   <gazebo reference="torso">
@@ -80,5 +81,5 @@
     <origin rpy="0 0 0" xyz="0.02 0 0.045" />
   </joint>
-  <xacro:mx28 name="mx28-head-pan" xyz="0 0 0" rpy="0 0 3.141592654"/>
+  <xacro:mx28 name="mx28-head-pan" x="0" y="0" z="0" rpy="0 0 3.141592654"/>
   <joint name="head-pan" type="revolute">
     <parent link="mx28-head-pan" />
@@ -90,14 +91,22 @@
   <link name="neck">
     <visual>
-      <origin rpy="0 0 0" xyz="0 0 0.03" />
-      <geometry>
-        <box size="0.01 0.01 0.01"/>
+      <origin rpy="0 0 0" xyz="0 0 0.02" />
+      <geometry>
+        <mesh filename="package://boldbot_description/meshes/neckbracketb.stl" scale="0.001 0.001 0.001"/>
       </geometry>
     </visual>
+    <collision>>
+      <origin rpy="0 0 0" xyz="0 0 0.02" />
+      <geometry>
+        <mesh filename="package://boldbot_description/meshes/neckbracketb.stl" scale="0.001 0.001 0.001"/>
+      </geometry>
+    </collision>
     <inertial>
-      <origin xyz="0 0 0" />
-      <xacro:xmass value="1e-3"/>
-      <inertia ixx="1e-4"  ixy="0.0"  ixz="0.0" iyy="1e-4" iyz="0.0" izz="1e-4" />
+      <origin xyz="0 0 0.029" />
+      <mass value="0.024357719"/>
+      <inertia ixx="0.0051411124"  ixy="-0.00057530255"  ixz="-0.000024729049" iyy="0.0081915737" iyz="-0.000019223094" izz="0.0011379812" />
     </inertial>
+    <!-- mass doubled to increase stability -->
+    <!-- <xacro:inertial_cuboid mass="0.025" xyz="0 0 0.029" x_length="0.025" y_length="0.045" z_length="0.0325" /> -->
   </link>
   <joint name="head-tilt" type="revolute">
@@ -108,5 +117,5 @@
     <limit effort="2.8" velocity="5.6548668" lower="-2.6179939" upper="2.6179939" />
   </joint>
-  <xacro:mx28 name="mx28-head-tilt" xyz="0 0 0" rpy="0 -1.570796327 -1.570796327"/>
+  <xacro:mx28 name="mx28-head-tilt" x="0" y="0" z="0" rpy="0 -1.570796327 -1.570796327"/>
   <joint name="head-tilt-head" type="fixed">
     <parent link="mx28-head-tilt" />
@@ -127,5 +136,5 @@
       </geometry>
     </collision>
-    <xacro:inertial_cuboid mass="0.2" xyz="0 0 0" x_length="0.05" y_length="0.1" z_length="0.04" />
+    <xacro:inertial_cuboid mass="0.2" xyz="0 0 0" rpy="0 0 0" x_length="0.05" y_length="0.1" z_length="0.04" />
   </link>
   <gazebo reference="head">
@@ -141,5 +150,5 @@
       <origin xyz="0.02 ${lr * 0.04} 0.045" />
     </joint>
-    <xacro:mx28 name="mx28-shoulder-pitch-${side}" xyz="0 0 0" rpy="${lr * 1.570796327} 0 3.141592654"/>
+    <xacro:mx28 name="mx28-shoulder-pitch-${side}" x="0" y="0" z="0" rpy="${lr * 1.570796327} 0 3.141592654"/>
     <joint name="shoulder-pitch-${side}" type="revolute">
       <parent link="mx28-shoulder-pitch-${side}" />
@@ -151,14 +160,15 @@
     <link name="shoulder-${side}">
       <visual>
-        <origin rpy="0 0 0" xyz="0 ${lr * 0.021} -0.008" />
-        <geometry>
-          <box size="0.01 0.01 0.01"/>
+        <origin rpy="0 0 ${0 if side == 'l' else 3.141592654}" xyz="0 ${lr * 0.02} 0" />
+        <geometry>
+          <mesh filename="package://boldbot_description/meshes/shoulderbracketb.stl" scale="0.001 0.001 0.001"/>
         </geometry>
       </visual>
       <inertial>
-        <origin xyz="0 0 0" />
-        <xacro:xmass value="0.1"/>
-        <inertia ixx="1e-4"  ixy="0.0"  ixz="0.0" iyy="1e-4" iyz="0.0" izz="1e-4" />
+        <origin xyz="0 ${lr * 0.038} -0.0025" />
+        <mass value="0.025913024"/>
+        <inertia ixx="0.0097758165"  ixy="0.0016911839"  ixz="-0.00045174329" iyx="0.0016911839" iyy="0.010511104" iyz="0.00033406955" izx="-0.00045174329" izy="0.00033406955" izz="0.005476798" />
       </inertial>
+      <!-- <xacro:inertial_cuboid mass="0.05" xyz="0 ${lr * 0.038} -0.0025" x_length="0.044" y_length="0.0332" z_length="0.038" /> -->
     </link>
     <joint name="shoulder-roll-${side}" type="revolute">
@@ -169,5 +179,5 @@
       <limit effort="2.8" velocity="5.6548668" lower="-2.6179939" upper="2.6179939" />
     </joint>
-    <xacro:mx28 name="mx28-shoulder-roll-${side}" xyz="0 0 0" rpy="0 1.570796327 0"/>
+    <xacro:mx28 name="mx28-shoulder-roll-${side}" x="0" y="0" z="0" rpy="0 1.570796327 0"/>
     <joint name="mx28-shoulder-roll-${side}-mx28-elbow-${side}" type="fixed">
       <parent link="mx28-shoulder-roll-${side}" />
@@ -175,5 +185,5 @@
       <origin xyz="0.016 0 -0.06" />
     </joint>
-    <xacro:mx28 name="mx28-elbow-${side}" xyz="0 0 0" rpy="${lr * 1.570796327} 0 3.141592654"/>
+    <xacro:mx28 name="mx28-elbow-${side}" x="0" y="0" z="0" rpy="${lr * 1.570796327} 0 3.141592654"/>
     <joint name="elbow-${side}" type="revolute">
       <parent link="mx28-elbow-${side}" />
@@ -196,9 +206,5 @@
         </geometry>
       </collision>
-      <inertial>
-        <origin xyz="0 0 0" />
-        <xacro:xmass value="0.1"/>
-        <inertia ixx="1e-3"  ixy="0.0"  ixz="0.0" iyy="1e-3" iyz="0.0" izz="1e-3" />
-      </inertial>
+      <xacro:inertial_cuboid mass="${2 * 0.000028534 * filament_density}" xyz="0.085 ${lr * 0.014} -0.02" rpy="${lr * 1.570796327} 0 0" x_length="0.1485" y_length="0.023" z_length="0.047" />
     </link>
     <gazebo reference="lower-arm-${side}">
@@ -217,5 +223,5 @@
       <origin xyz="0.018 ${lr * 0.037} -0.04" />
     </joint>
-    <xacro:mx28 name="mx28-hip-yaw-${side}" xyz="0 0 0" rpy="${lr * 3.141592654} 0 3.141592654"/>
+    <xacro:mx28 name="mx28-hip-yaw-${side}" x="0" y="0" z="0" rpy="${lr * 3.141592654} 0 3.141592654"/>
     <joint name="hip-yaw-${side}" type="revolute">
       <parent link="mx28-hip-yaw-${side}" />
@@ -227,6 +233,6 @@
     <link name="hip-bracket-${side}">
       <inertial>
-        <origin xyz="0 0 0" />
-        <xacro:xmass value=".1"/>
+        <origin xyz="0 0 -0.02" />
+        <xacro:xmass value="0.025"/>
         <inertia ixx="1e-4"  ixy="0.0"  ixz="0.0" iyy="1e-4" iyz="0.0" izz="1e-4" />
       </inertial>
@@ -239,5 +245,5 @@
       <limit effort="2.8" velocity="5.6548668" lower="-2.6179939" upper="2.6179939" />
     </joint>
-    <xacro:mx28 name="mx28-hip-roll-${side}" xyz="0 0 0" rpy="0 1.570796327 0"/>
+    <xacro:mx28 name="mx28-hip-roll-${side}" x="0" y="0" z="0" rpy="0 1.570796327 0"/>
     <joint name="mx28-hip-roll-mx28-hip-pitch-${side}" type="fixed">
       <parent link="mx28-hip-roll-${side}" />
@@ -245,5 +251,5 @@
       <origin xyz="0.05 0 0" rpy="0 0 0" />
     </joint>
-    <xacro:mx28 name="mx28-hip-pitch-${side}" xyz="0 0 0" rpy="1.570796327 1.570796327 0"/>
+    <xacro:mx28 name="mx28-hip-pitch-${side}" x="0" y="0" z="0" rpy="1.570796327 1.570796327 0"/>
     <joint name="hip-pitch-${side}" type="revolute">
       <parent link="mx28-hip-pitch-${side}" />
@@ -266,9 +272,6 @@
         </geometry>
       </collision>
-      <inertial>
-        <origin xyz="0 0 0" />
-        <xacro:xmass value="0.1"/>
-        <inertia ixx="1e-3"  ixy="0.0"  ixz="0.0" iyy="1e-3" iyz="0.0" izz="1e-3" />
-      </inertial>
+      <!-- Mass and COM measured with Meshlab -->
+      <xacro:inertial_cuboid mass="${0.000051158 * filament_density}" xyz="0 0 -0.067" rpy="0 1.570796327 0" x_length="0.025" y_length="0.0515" z_length="0.117" />
     </link>
     <gazebo reference="upper-leg-${side}">
@@ -281,5 +284,5 @@
       <origin xyz="0 0 -0.143" rpy="0 0 0" />
     </joint>
-    <xacro:mx28 name="mx28-knee-${side}" xyz="0 0 0" rpy="1.570796327 -1.570796327 0"/>
+    <xacro:mx28 name="mx28-knee-${side}" x="0" y="0" z="0" rpy="1.570796327 -1.570796327 0"/>
     <joint name="knee-${side}" type="revolute">
       <parent link="mx28-knee-${side}" />
@@ -302,9 +305,6 @@
         </geometry>
       </collision>
-      <inertial>
-	<origin xyz="0 0 0" />
-	<mass value="0.1"/>
-	<inertia ixx="1e-3"  ixy="0.0"  ixz="0.0" iyy="1e-3" iyz="0.0" izz="1e-3" />
-      </inertial>
+      <!-- Mass and COM measured with Meshlab -->
+      <xacro:inertial_cuboid mass="${0.000055347 * filament_density}" xyz="0.013 0 -0.055" rpy="3.141592654 1.570796327 0" x_length="0.042" y_length="0.051" z_length="0.1555" />
     </link>
     <gazebo reference="lower-leg-${side}">
@@ -319,5 +319,5 @@
       <limit effort="2.8" velocity="5.6548668" lower="-2.6179939" upper="2.6179939" />
     </joint>
-    <xacro:mx28 name="mx28-ankle-pitch-${side}" xyz="0 0 0" rpy="1.570796327 -1.570796327 0"/>
+    <xacro:mx28 name="mx28-ankle-pitch-${side}" x="0" y="0" z="0" rpy="1.570796327 -1.570796327 0"/>
     <joint name="mx28-ankle-pitch-mx28-ankle-roll-${side}" type="fixed">
       <parent link="mx28-ankle-pitch-${side}" />
@@ -325,5 +325,5 @@
       <origin xyz="-0.05 0 0" rpy="0 0 0" />
     </joint>
-    <xacro:mx28 name="mx28-ankle-roll-${side}" xyz="0 0 0" rpy="3.141592654 -1.570796327 0"/>
+    <xacro:mx28 name="mx28-ankle-roll-${side}" x="0" y="0" z="0" rpy="3.141592654 -1.570796327 0"/>
     <joint name="ankle-roll-${side}" type="revolute">
       <parent link="mx28-ankle-roll-${side}" />

Commit message: Pass on coordinates through macros

File: boldbot_description/urdf/boldbot.urdf.xacro (robot description, xacro)
@@ -11,5 +11,5 @@
     <inertial>
       <xacro:xmass value="${mass}" />
-      <origin rpy="0 0 0" xyz="${xyz}"/>
+      <origin rpy="${rpy}" xyz="${xyz}"/>
       <inertia ixx="${mass * (y_length*y_length + z_length*z_length) / 12}" ixy="0.0" ixz="0.0"
                iyy="${mass * (x_length*x_length + z_length*z_length) / 12}" iyz="0.0"
@@ -26,8 +26,8 @@
   <!--   </inertial> -->
   <!-- </xacro:macro> -->
-  <xacro:macro name="mx28" params="name">
+  <xacro:macro name="mx28" params="name x y z rpy">
     <link name="${name}">
       <visual>
-        <origin xyz="0 0 0" rpy="0 0 0" />
+        <origin xyz="${x} ${y} ${z}" rpy="${rpy}" />
         <geometry>
           <mesh filename="package://boldbot_description/meshes/mx28b.stl" scale="0.001 0.001 0.001" />
@@ -38,10 +38,10 @@
       </visual>
       <collision>
-        <origin xyz="0 0 0" rpy="0 0 0" />
+        <origin xyz="${x} ${y} ${z}" rpy="${rpy}" />
         <geometry>
           <mesh filename="package://boldbot_description/meshes/mx28b.stl" scale="0.001 0.001 0.001" />
         </geometry>
       </collision>
-      <xacro:inertial_cuboid mass="0.077" xyz="0.0105 0 0" rpy="0 0 0" x_length="0.0506" y_length="0.0356" z_length="0.0355" />
+      <xacro:inertial_cuboid mass="0.077" xyz="${x + 0.0105} ${y} ${z}" rpy="${rpy}" x_length="0.0506" y_length="0.0356" z_length="0.0355" />
     </link>
     <gazebo reference="${name}">
